Commit message: robot simulation still not working

File: src/robot_description/urdf/robot.urdf.xacro (robot description, xacro)
@@ -14,5 +14,5 @@
       <origin xyz="1.67553 -2.50292 1.41602" rpy="0 -0 0"/>
       <geometry>
-        <mesh filename="package://assets/v_slot_20x40x1500_linear_rail.stl"/>
+        <mesh filename="package://robot_description/meshes/v_slot_20x40x1500_linear_rail.stl"/>
       </geometry>
       <material name="v_slot_20x40x1500_linear_rail_material">
@@ -23,5 +23,5 @@
       <origin xyz="1.67553 -2.50292 1.41602" rpy="0 -0 0"/>
       <geometry>
-        <mesh filename="package://assets/v_slot_20x40x1500_linear_rail.stl"/>
+        <mesh filename="package://robot_description/meshes/v_slot_20x40x1500_linear_rail.stl"/>
       </geometry>
     </collision>
@@ -30,5 +30,5 @@
       <origin xyz="0.190533 -1.00292 1.41602" rpy="0 -0 0"/>
       <geometry>
-        <mesh filename="package://assets/v_slot_20x40x1500_linear_rail.stl"/>
+        <mesh filename="package://robot_description/meshes/v_slot_20x40x1500_linear_rail.stl"/>
       </geometry>
       <material name="v_slot_20x40x1500_linear_rail_2_material">
@@ -39,5 +39,5 @@
       <origin xyz="0.190533 -1.00292 1.41602" rpy="0 -0 0"/>
       <geometry>
-        <mesh filename="package://assets/v_slot_20x40x1500_linear_rail.stl"/>
+        <mesh filename="package://robot_description/meshes/v_slot_20x40x1500_linear_rail.stl"/>
       </geometry>
     </collision>
@@ -46,5 +46,5 @@
       <origin xyz="0.190533 -2.50292 1.41602" rpy="0 -0 0"/>
       <geometry>
-        <mesh filename="package://assets/v_slot_20x40x1500_linear_rail.stl"/>
+        <mesh filename="package://robot_description/meshes/v_slot_20x40x1500_linear_rail.stl"/>
       </geometry>
       <material name="v_slot_20x40x1500_linear_rail_3_material">
@@ -55,5 +55,5 @@
       <origin xyz="0.190533 -2.50292 1.41602" rpy="0 -0 0"/>
       <geometry>
-        <mesh filename="package://assets/v_slot_20x40x1500_linear_rail.stl"/>
+        <mesh filename="package://robot_description/meshes/v_slot_20x40x1500_linear_rail.stl"/>
       </geometry>
     </collision>
@@ -62,5 +62,5 @@
       <origin xyz="1.67553 -1.00292 1.41602" rpy="0 -0 0"/>
       <geometry>
-        <mesh filename="package://assets/v_slot_20x40x1500_linear_rail.stl"/>
+        <mesh filename="package://robot_description/meshes/v_slot_20x40x1500_linear_rail.stl"/>
       </geometry>
       <material name="v_slot_20x40x1500_linear_rail_4_material">
@@ -71,5 +71,5 @@
       <origin xyz="1.67553 -1.00292 1.41602" rpy="0 -0 0"/>
       <geometry>
-        <mesh filename="package://assets/v_slot_20x40x1500_linear_rail.stl"/>
+        <mesh filename="package://robot_description/meshes/v_slot_20x40x1500_linear_rail.stl"/>
       </geometry>
     </collision>
@@ -78,5 +78,5 @@
       <origin xyz="1.68953 -2.50352 1.40652" rpy="-1.5708 -0 1.5708"/>
       <geometry>
-        <mesh filename="package://assets/joining_plate_t.stl"/>
+        <mesh filename="package://robot_description/meshes/joining_plate_t.stl"/>
       </geometry>
       <material name="joining_plate_t_material">
@@ -87,5 +87,5 @@
       <origin xyz="1.68953 -2.50352 1.40652" rpy="-1.5708 -0 1.5708"/>
       <geometry>
-        <mesh filename="package://assets/joining_plate_t.stl"/>
+        <mesh filename="package://robot_description/meshes/joining_plate_t.stl"/>
       </geometry>
     </collision>
@@ -94,5 +94,5 @@
       <origin xyz="0.176533 -2.50295 1.40652" rpy="-1.5708 0 -1.5708"/>
       <geometry>
-        <mesh filename="package://assets/joining_plate_t.stl"/>
+        <mesh filename="package://robot_description/meshes/joining_plate_t.stl"/>
       </geometry>
       <material name="joining_plate_t_2_material">
@@ -103,5 +103,5 @@
       <origin xyz="0.176533 -2.50295 1.40652" rpy="-1.5708 0 -1.5708"/>
       <geometry>
-        <mesh filename="package://assets/joining_plate_t.stl"/>
+        <mesh filename="package://robot_description/meshes/joining_plate_t.stl"/>
       </geometry>
     </collision>
@@ -110,5 +110,5 @@
       <origin xyz="0.180533 -1.01292 1.40652" rpy="-1.5708 -0 1.5708"/>
       <geometry>
-        <mesh filename="package://assets/joining_plate_90_degree.stl"/>
+        <mesh filename="package://robot_description/meshes/joining_plate_90_degree.stl"/>
       </geometry>
       <material name="joining_plate_90_degree_material">
@@ -119,5 +119,5 @@
       <origin xyz="0.180533 -1.01292 1.40652" rpy="-1.5708 -0 1.5708"/>
       <geometry>
-        <mesh filename="package://assets/joining_plate_90_degree.stl"/>
+        <mesh filename="package://robot_description/meshes/joining_plate_90_degree.stl"/>
       </geometry>
     </collision>
@@ -126,5 +126,5 @@
       <origin xyz="0.176533 -3.99292 1.40652" rpy="-1.5708 -0 -1.5708"/>
       <geometry>
-        <mesh filename="package://assets/joining_plate_90_degree.stl"/>
+        <mesh filename="package://robot_description/meshes/joining_plate_90_degree.stl"/>
       </geometry>
       <material name="joining_plate_90_degree_2_material">
@@ -135,5 +135,5 @@
       <origin xyz="0.176533 -3.99292 1.40652" rpy="-1.5708 -0 -1.5708"/>
       <geometry>
-        <mesh filename="package://assets/joining_plate_90_degree.stl"/>
+        <mesh filename="package://robot_description/meshes/joining_plate_90_degree.stl"/>
       </geometry>
     </collision>
@@ -142,5 +142,5 @@
       <origin xyz="1.66153 -3.99292 1.40652" rpy="-1.5708 -0 -1.5708"/>
       <geometry>
-        <mesh filename="package://assets/joining_plate_90_degree.stl"/>
+        <mesh filename="package://robot_description/meshes/joining_plate_90_degree.stl"/>
       </geometry>
       <material name="joining_plate_90_degree_3_material">
@@ -151,5 +151,5 @@
       <origin xyz="1.66153 -3.99292 1.40652" rpy="-1.5708 -0 -1.5708"/>
       <geometry>
-        <mesh filename="package://assets/joining_plate_90_degree.stl"/>
+        <mesh filename="package://robot_description/meshes/joining_plate_90_degree.stl"/>
       </geometry>
     </collision>
@@ -158,5 +158,5 @@
       <origin xyz="1.68953 -1.01292 1.40652" rpy="-1.5708 -0 1.5708"/>
       <geometry>
-        <mesh filename="package://assets/joining_plate_90_degree.stl"/>
+        <mesh filename="package://robot_description/meshes/joining_plate_90_degree.stl"/>
       </geometry>
       <material name="joining_plate_90_degree_4_material">
@@ -167,5 +167,5 @@
       <origin xyz="1.68953 -1.01292 1.40652" rpy="-1.5708 -0 1.5708"/>
       <geometry>
-        <mesh filename="package://assets/joining_plate_90_degree.stl"/>
+        <mesh filename="package://robot_description/meshes/joining_plate_90_degree.stl"/>
       </geometry>
     </collision>
@@ -174,5 +174,5 @@
       <origin xyz="1.66553 -1.01292 1.40652" rpy="-1.5708 -0 1.5708"/>
       <geometry>
-        <mesh filename="package://assets/joining_plate_90_degree.stl"/>
+        <mesh filename="package://robot_description/meshes/joining_plate_90_degree.stl"/>
       </geometry>
       <material name="joining_plate_90_degree_5_material">
@@ -183,5 +183,5 @@
       <origin xyz="1.66553 -1.01292 1.40652" rpy="-1.5708 -0 1.5708"/>
       <geometry>
-        <mesh filename="package://assets/joining_plate_90_degree.stl"/>
+        <mesh filename="package://robot_description/meshes/joining_plate_90_degree.stl"/>
       </geometry>
     </collision>
@@ -190,5 +190,5 @@
       <origin xyz="0.200533 -3.99292 1.40652" rpy="-1.5708 -0 -1.5708"/>
       <geometry>
-        <mesh filename="package://assets/joining_plate_90_degree.stl"/>
+        <mesh filename="package://robot_description/meshes/joining_plate_90_degree.stl"/>
       </geometry>
       <material name="joining_plate_90_degree_6_material">
@@ -199,5 +199,5 @@
       <origin xyz="0.200533 -3.99292 1.40652" rpy="-1.5708 -0 -1.5708"/>
       <geometry>
-        <mesh filename="package://assets/joining_plate_90_degree.stl"/>
+        <mesh filename="package://robot_description/meshes/joining_plate_90_degree.stl"/>
       </geometry>
     </collision>
@@ -206,5 +206,5 @@
       <origin xyz="0.204533 -1.01292 1.40652" rpy="-1.5708 -0 1.5708"/>
       <geometry>
-        <mesh filename="package://assets/joining_plate_90_degree.stl"/>
+        <mesh filename="package://robot_description/meshes/joining_plate_90_degree.stl"/>
       </geometry>
       <material name="joining_plate_90_degree_7_material">
@@ -215,5 +215,5 @@
       <origin xyz="0.204533 -1.01292 1.40652" rpy="-1.5708 -0 1.5708"/>
       <geometry>
-        <mesh filename="package://assets/joining_plate_90_degree.stl"/>
+        <mesh filename="package://robot_description/meshes/joining_plate_90_degree.stl"/>
       </geometry>
     </collision>
@@ -222,5 +222,5 @@
       <origin xyz="1.68553 -3.99292 1.40652" rpy="-1.5708 -0 -1.5708"/>
       <geometry>
-        <mesh filename="package://assets/joining_plate_90_degree.stl"/>
+        <mesh filename="package://robot_description/meshes/joining_plate_90_degree.stl"/>
       </geometry>
       <material name="joining_plate_90_degree_8_material">
@@ -231,5 +231,5 @@
       <origin xyz="1.68553 -3.99292 1.40652" rpy="-1.5708 -0 -1.5708"/>
       <geometry>
-        <mesh filename="package://assets/joining_plate_90_degree.stl"/>
+        <mesh filename="package://robot_description/meshes/joining_plate_90_degree.stl"/>
       </geometry>
     </collision>
@@ -238,5 +238,5 @@
       <origin xyz="1.68023 -2.50352 1.40652" rpy="-1.5708 1.5708 0"/>
       <geometry>
-        <mesh filename="package://assets/m5_tee_nut.stl"/>
+        <mesh filename="package://robot_description/meshes/m5_tee_nut.stl"/>
       </geometry>
       <material name="m5_tee_nut_material">
@@ -247,5 +247,5 @@
       <origin xyz="1.68023 -2.50352 1.40652" rpy="-1.5708 1.5708 0"/>
       <geometry>
-        <mesh filename="package://assets/m5_tee_nut.stl"/>
+        <mesh filename="package://robot_description/meshes/m5_tee_nut.stl"/>
       </geometry>
     </collision>
@@ -254,5 +254,5 @@
       <origin xyz="1.68953 -2.50352 1.40652" rpy="-1.5708 1.5708 0"/>
       <geometry>
-        <mesh filename="package://assets/m5_x_10mm_screw.stl"/>
+        <mesh filename="package://robot_description/meshes/m5_x_10mm_screw.stl"/>
       </geometry>
       <material name="m5_x_10mm_screw_material">
@@ -263,5 +263,5 @@
       <origin xyz="1.68953 -2.50352 1.40652" rpy="-1.5708 1.5708 0"/>
       <geometry>
-        <mesh filename="package://assets/m5_x_10mm_screw.stl"/>
+        <mesh filename="package://robot_description/meshes/m5_x_10mm_screw.stl"/>
       </geometry>
     </collision>
@@ -270,5 +270,5 @@
       <origin xyz="1.68023 -2.48352 1.40652" rpy="-1.5708 1.5708 0"/>
       <geometry>
-        <mesh filename="package://assets/m5_tee_nut.stl"/>
+        <mesh filename="package://robot_description/meshes/m5_tee_nut.stl"/>
       </geometry>
       <material name="m5_tee_nut_2_material">
@@ -279,5 +279,5 @@
       <origin xyz="1.68023 -2.48352 1.40652" rpy="-1.5708 1.5708 0"/>
       <geometry>
-        <mesh filename="package://assets/m5_tee_nut.stl"/>
+        <mesh filename="package://robot_description/meshes/m5_tee_nut.stl"/>
       </geometry>
     </collision>
@@ -286,5 +286,5 @@
       <origin xyz="1.68953 -2.48352 1.40652" rpy="-1.5708 1.5708 0"/>
       <geometry>
-        <mesh filename="package://assets/m5_x_10mm_screw.stl"/>
+        <mesh filename="package://robot_description/meshes/m5_x_10mm_screw.stl"/>
       </geometry>
       <material name="m5_x_10mm_screw_2_material">
@@ -295,5 +295,5 @@
       <origin xyz="1.68953 -2.48352 1.40652" rpy="-1.5708 1.5708 0"/>
       <geometry>
-        <mesh filename="package://assets/m5_x_10mm_screw.stl"/>
+        <mesh filename="package://robot_description/meshes/m5_x_10mm_screw.stl"/>
       </geometry>
     </collision>
@@ -302,5 +302,5 @@
       <origin xyz="1.68023 -2.52352 1.40652" rpy="-1.5708 1.5708 0"/>
       <geometry>
-        <mesh filename="package://assets/m5_tee_nut.stl"/>
+        <mesh filename="package://robot_description/meshes/m5_tee_nut.stl"/>
       </geometry>
       <material name="m5_tee_nut_3_material">
@@ -311,5 +311,5 @@
       <origin xyz="1.68023 -2.52352 1.40652" rpy="-1.5708 1.5708 0"/>
       <geometry>
-        <mesh filename="package://assets/m5_tee_nut.stl"/>
+        <mesh filename="package://robot_description/meshes/m5_tee_nut.stl"/>
       </geometry>
     </collision>
@@ -318,5 +318,5 @@
       <origin xyz="1.68953 -2.52352 1.40652" rpy="-1.5708 1.5708 0"/>
       <geometry>
-        <mesh filename="package://assets/m5_x_10mm_screw.stl"/>
+        <mesh filename="package://robot_description/meshes/m5_x_10mm_screw.stl"/>
       </geometry>
       <material name="m5_x_10mm_screw_3_material">
@@ -327,5 +327,5 @@
       <origin xyz="1.68953 -2.52352 1.40652" rpy="-1.5708 1.5708 0"/>
       <geometry>
-        <mesh filename="package://assets/m5_x_10mm_screw.stl"/>
+        <mesh filename="package://robot_description/meshes/m5_x_10mm_screw.stl"/>
       </geometry>
     </collision>
@@ -334,5 +334,5 @@
       <origin xyz="0.185833 -2.50295 1.40652" rpy="1.5708 1.5708 0"/>
       <geometry>
-        <mesh filename="package://assets/m5_tee_nut.stl"/>
+        <mesh filename="package://robot_description/meshes/m5_tee_nut.stl"/>
       </geometry>
       <material name="m5_tee_nut_4_material">
@@ -343,5 +343,5 @@
       <origin xyz="0.185833 -2.50295 1.40652" rpy="1.5708 1.5708 0"/>
       <geometry>
-        <mesh filename="package://assets/m5_tee_nut.stl"/>
+        <mesh filename="package://robot_description/meshes/m5_tee_nut.stl"/>
       </geometry>
     </collision>
@@ -350,5 +350,5 @@
       <origin xyz="0.176533 -2.50295 1.40652" rpy="1.5708 1.5708 0"/>
       <geometry>
-        <mesh filename="package://assets/m5_x_10mm_screw.stl"/>
+        <mesh filename="package://robot_description/meshes/m5_x_10mm_screw.stl"/>
       </geometry>
       <material name="m5_x_10mm_screw_4_material">
@@ -359,5 +359,5 @@
       <origin xyz="0.176533 -2.50295 1.40652" rpy="1.5708 1.5708 0"/>
       <geometry>
-        <mesh filename="package://assets/m5_x_10mm_screw.stl"/>
+        <mesh filename="package://robot_description/meshes/m5_x_10mm_screw.stl"/>
       </geometry>
     </collision>
@@ -366,5 +366,5 @@
       <origin xyz="0.185833 -2.52295 1.40652" rpy="1.5708 1.5708 0"/>
       <geometry>
-        <mesh filename="package://assets/m5_tee_nut.stl"/>
+        <mesh filename="package://robot_description/meshes/m5_tee_nut.stl"/>
       </geometry>
       <material name="m5_tee_nut_5_material">
@@ -375,5 +375,5 @@
       <origin xyz="0.185833 -2.52295 1.40652" rpy="1.5708 1.5708 0"/>
       <geometry>
-        <mesh filename="package://assets/m5_tee_nut.stl"/>
+        <mesh filename="package://robot_description/meshes/m5_tee_nut.stl"/>
       </geometry>
     </collision>
@@ -382,5 +382,5 @@
       <origin xyz="0.176533 -2.52295 1.40652" rpy="1.5708 1.5708 0"/>
       <geometry>
-        <mesh filename="package://assets/m5_x_10mm_screw.stl"/>
+        <mesh filename="package://robot_description/meshes/m5_x_10mm_screw.stl"/>
       </geometry>
       <material name="m5_x_10mm_screw_5_material">
@@ -391,5 +391,5 @@
       <origin xyz="0.176533 -2.52295 1.40652" rpy="1.5708 1.5708 0"/>
       <geometry>
-        <mesh filename="package://assets/m5_x_10mm_screw.stl"/>
+        <mesh filename="package://robot_description/meshes/m5_x_10mm_screw.stl"/>
       </geometry>
     </collision>
@@ -398,5 +398,5 @@
       <origin xyz="0.185833 -2.48295 1.40652" rpy="1.5708 1.5708 0"/>
       <geometry>
-        <mesh filename="package://assets/m5_tee_nut.stl"/>
+        <mesh filename="package://robot_description/meshes/m5_tee_nut.stl"/>
       </geometry>
       <material name="m5_tee_nut_6_material">
@@ -407,5 +407,5 @@
       <origin xyz="0.185833 -2.48295 1.40652" rpy="1.5708 1.5708 0"/>
       <geometry>
-        <mesh filename="package://assets/m5_tee_nut.stl"/>
+        <mesh filename="package://robot_description/meshes/m5_tee_nut.stl"/>
       </geometry>
     </collision>
@@ -414,5 +414,5 @@
       <origin xyz="0.176533 -2.48295 1.40652" rpy="1.5708 1.5708 0"/>
       <geometry>
-        <mesh filename="package://assets/m5_x_10mm_screw.stl"/>
+        <mesh filename="package://robot_description/meshes/m5_x_10mm_screw.stl"/>
       </geometry>
       <material name="m5_x_10mm_screw_6_material">
@@ -423,5 +423,5 @@
       <origin xyz="0.176533 -2.48295 1.40652" rpy="1.5708 1.5708 0"/>
       <geometry>
-        <mesh filename="package://assets/m5_x_10mm_screw.stl"/>
+        <mesh filename="package://robot_description/meshes/m5_x_10mm_screw.stl"/>
       </geometry>
     </collision>
@@ -430,5 +430,5 @@
       <origin xyz="0.185833 -1.03292 1.40652" rpy="3.14159 -0 1.5708"/>
       <geometry>
-        <mesh filename="package://assets/m5_tee_nut.stl"/>
+        <mesh filename="package://robot_description/meshes/m5_tee_nut.stl"/>
       </geometry>
       <material name="m5_tee_nut_7_material">
@@ -439,5 +439,5 @@
       <origin xyz="0.185833 -1.03292 1.40652" rpy="3.14159 -0 1.5708"/>
       <geometry>
-        <mesh filename="package://assets/m5_tee_nut.stl"/>
+        <mesh filename="package://robot_description/meshes/m5_tee_nut.stl"/>
       </geometry>
     </collision>
@@ -446,5 +446,5 @@
       <origin xyz="0.176533 -1.03292 1.40652" rpy="3.14159 -0 1.5708"/>
       <geometry>
-        <mesh filename="package://assets/m5_x_10mm_screw.stl"/>
+        <mesh filename="package://robot_description/meshes/m5_x_10mm_screw.stl"/>
       </geometry>
       <material name="m5_x_10mm_screw_7_material">
@@ -455,5 +455,5 @@
       <origin xyz="0.176533 -1.03292 1.40652" rpy="3.14159 -0 1.5708"/>
       <geometry>
-        <mesh filename="package://assets/m5_x_10mm_screw.stl"/>
+        <mesh filename="package://robot_description/meshes/m5_x_10mm_screw.stl"/>
       </geometry>
     </collision>
@@ -462,5 +462,5 @@
       <origin xyz="0.185833 -1.05292 1.40652" rpy="3.14159 -0 1.5708"/>
       <geometry>
-        <mesh filename="package://assets/m5_tee_nut.stl"/>
+        <mesh filename="package://robot_description/meshes/m5_tee_nut.stl"/>
       </geometry>
       <material name="m5_tee_nut_8_material">
@@ -471,5 +471,5 @@
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