Commit message: updated robot description

File: src/robot_description/urdf/robot.urdf.xacro (robot description, xacro)
@@ -1,1197 +1,9949 @@
-<?xml version="1.0" ?>
+<?xml version="1.0"?>
 <!-- Generated using onshape-to-robot -->
-<!-- Onshape https://cad.onshape.com/documents/30d6379e78de76482470e7ee/w/e7b346f4bf0df2c360371a5c/e/263883c8752f9c1b548bfc82 -->
+<!-- Onshape
+https://cad.onshape.com/documents/a2e4d90d4720e7eb81b47647/w/f29fb00f1617a93c8228a45a/e/cddef7938b795a6053ad7145 -->
 <robot name="surgeyos-robot2">
   <!-- Link x_axis_tracks -->
-  <link name="x_axis_tracks">
+  <link name="x_axis_tracks_inertial">
     <inertial>
-      <origin xyz="0 0 0" rpy="0 0 0"/>
-      <mass value="1e-09"/>
-      <inertia ixx="1e-09" ixy="0" ixz="0" iyy="1e-09" iyz="0" izz="1e-09"/>
+      <origin xyz="0 0 0" rpy="0 0 0" />
+      <mass value="1e-09" />
+      <inertia ixx="1e-09" ixy="0" ixz="0" iyy="1e-09" iyz="0" izz="1e-09" />
     </inertial>
-    <!-- Part v_slot_20x40x1500_linear_rail -->
-    <visual>
-      <origin xyz="1.67553 -2.50292 1.41602" rpy="0 -0 0"/>
-      <geometry>
-        <mesh filename="package://robot_description/meshes/v_slot_20x40x1500_linear_rail.stl"/>
+  </link>
+  <!-- Part v_slot_20x40x1500_linear_rail -->
+  <link name="v_slot_20x40x1500_linear_rail">
+    <visual>
+      <origin xyz="1.67553 -2.50292 1.41602" rpy="0 -0 0" />
+      <geometry>
+        <mesh filename="./assets/v_slot_20x40x1500_linear_rail.stl" />
       </geometry>
       <material name="v_slot_20x40x1500_linear_rail_material">
-        <color rgba="0.866667 0.909804 1 1"/>
-      </material>
-    </visual>
-    <collision>
-      <origin xyz="1.67553 -2.50292 1.41602" rpy="0 -0 0"/>
-      <geometry>
-        <mesh filename="package://robot_description/meshes/v_slot_20x40x1500_linear_rail.stl"/>
-      </geometry>
-    </collision>
-    <!-- Part v_slot_20x40x1500_linear_rail_2 -->
-    <visual>
-      <origin xyz="0.190533 -1.00292 1.41602" rpy="0 -0 0"/>
-      <geometry>
-        <mesh filename="package://robot_description/meshes/v_slot_20x40x1500_linear_rail.stl"/>
+        <color rgba="0.866667 0.909804 1 1" />
+      </material>
+    </visual>
+    <collision>
+      <origin xyz="1.67553 -2.50292 1.41602" rpy="0 -0 0" />
+      <geometry>
+        <mesh filename="./assets/v_slot_20x40x1500_linear_rail.stl" />
+      </geometry>
+    </collision>
+  </link>
+  <!-- Part v_slot_20x40x1500_linear_rail_2 -->
+  <link name="v_slot_20x40x1500_linear_rail_2">
+    <visual>
+      <origin xyz="0.190533 -1.00292 1.41602" rpy="0 -0 0" />
+      <geometry>
+        <mesh filename="./assets/v_slot_20x40x1500_linear_rail.stl" />
       </geometry>
       <material name="v_slot_20x40x1500_linear_rail_2_material">
-        <color rgba="0.866667 0.909804 1 1"/>
-      </material>
-    </visual>
-    <collision>
-      <origin xyz="0.190533 -1.00292 1.41602" rpy="0 -0 0"/>
-      <geometry>
-        <mesh filename="package://robot_description/meshes/v_slot_20x40x1500_linear_rail.stl"/>
-      </geometry>
-    </collision>
-    <!-- Part v_slot_20x40x1500_linear_rail_3 -->
-    <visual>
-      <origin xyz="0.190533 -2.50292 1.41602" rpy="0 -0 0"/>
-      <geometry>
-        <mesh filename="package://robot_description/meshes/v_slot_20x40x1500_linear_rail.stl"/>
+        <color rgba="0.866667 0.909804 1 1" />
+      </material>
+    </visual>
+    <collision>
+      <origin xyz="0.190533 -1.00292 1.41602" rpy="0 -0 0" />
+      <geometry>
+        <mesh filename="./assets/v_slot_20x40x1500_linear_rail.stl" />
+      </geometry>
+    </collision>
+  </link>
+  <!-- Part v_slot_20x40x1500_linear_rail_3 -->
+  <link name="v_slot_20x40x1500_linear_rail_3">
+    <visual>
+      <origin xyz="0.190533 -2.50292 1.41602" rpy="0 -0 0" />
+      <geometry>
+        <mesh filename="./assets/v_slot_20x40x1500_linear_rail.stl" />
       </geometry>
       <material name="v_slot_20x40x1500_linear_rail_3_material">
-        <color rgba="0.866667 0.909804 1 1"/>
-      </material>
-    </visual>
-    <collision>
-      <origin xyz="0.190533 -2.50292 1.41602" rpy="0 -0 0"/>
-      <geometry>
-        <mesh filename="package://robot_description/meshes/v_slot_20x40x1500_linear_rail.stl"/>
-      </geometry>
-    </collision>
-    <!-- Part v_slot_20x40x1500_linear_rail_4 -->
-    <visual>
-      <origin xyz="1.67553 -1.00292 1.41602" rpy="0 -0 0"/>
-      <geometry>
-        <mesh filename="package://robot_description/meshes/v_slot_20x40x1500_linear_rail.stl"/>
+        <color rgba="0.866667 0.909804 1 1" />
+      </material>
+    </visual>
+    <collision>
+      <origin xyz="0.190533 -2.50292 1.41602" rpy="0 -0 0" />
+      <geometry>
+        <mesh filename="./assets/v_slot_20x40x1500_linear_rail.stl" />
+      </geometry>
+    </collision>
+  </link>
+  <!-- Part v_slot_20x40x1500_linear_rail_4 -->
+  <link name="v_slot_20x40x1500_linear_rail_4">
+    <visual>
+      <origin xyz="1.67553 -1.00292 1.41602" rpy="0 -0 0" />
+      <geometry>
+        <mesh filename="./assets/v_slot_20x40x1500_linear_rail.stl" />
       </geometry>
       <material name="v_slot_20x40x1500_linear_rail_4_material">
-        <color rgba="0.866667 0.909804 1 1"/>
-      </material>
-    </visual>
-    <collision>
-      <origin xyz="1.67553 -1.00292 1.41602" rpy="0 -0 0"/>
-      <geometry>
-        <mesh filename="package://robot_description/meshes/v_slot_20x40x1500_linear_rail.stl"/>
-      </geometry>
-    </collision>
-    <!-- Part joining_plate_t -->
-    <visual>
-      <origin xyz="1.68953 -2.50352 1.40652" rpy="-1.5708 -0 1.5708"/>
-      <geometry>
-        <mesh filename="package://robot_description/meshes/joining_plate_t.stl"/>
+        <color rgba="0.866667 0.909804 1 1" />
+      </material>
+    </visual>
+    <collision>
+      <origin xyz="1.67553 -1.00292 1.41602" rpy="0 -0 0" />
+      <geometry>
+        <mesh filename="./assets/v_slot_20x40x1500_linear_rail.stl" />
+      </geometry>
+    </collision>
+  </link>
+  <!-- Part joining_plate_t -->
+  <link name="joining_plate_t">
+    <visual>
+      <origin xyz="1.68953 -2.50352 1.40652" rpy="-1.5708 -0 1.5708" />
+      <geometry>
+        <mesh filename="./assets/joining_plate_t.stl" />
       </geometry>
       <material name="joining_plate_t_material">
-        <color rgba="0.866667 0.909804 1 1"/>
-      </material>
-    </visual>
-    <collision>
-      <origin xyz="1.68953 -2.50352 1.40652" rpy="-1.5708 -0 1.5708"/>
-      <geometry>
-        <mesh filename="package://robot_description/meshes/joining_plate_t.stl"/>
-      </geometry>
-    </collision>
-    <!-- Part joining_plate_t_2 -->
-    <visual>
-      <origin xyz="0.176533 -2.50295 1.40652" rpy="-1.5708 0 -1.5708"/>
-      <geometry>
-        <mesh filename="package://robot_description/meshes/joining_plate_t.stl"/>
+        <color rgba="0.866667 0.909804 1 1" />
+      </material>
+    </visual>
+    <collision>
+      <origin xyz="1.68953 -2.50352 1.40652" rpy="-1.5708 -0 1.5708" />
+      <geometry>
+        <mesh filename="./assets/joining_plate_t.stl" />
+      </geometry>
+    </collision>
+  </link>
+  <!-- Part joining_plate_t_2 -->
+  <link name="joining_plate_t_2">
+    <visual>
+      <origin xyz="0.176533 -2.50295 1.40652" rpy="-1.5708 0 -1.5708" />
+      <geometry>
+        <mesh filename="./assets/joining_plate_t.stl" />
       </geometry>
       <material name="joining_plate_t_2_material">
-        <color rgba="0.866667 0.909804 1 1"/>
-      </material>
-    </visual>
-    <collision>
-      <origin xyz="0.176533 -2.50295 1.40652" rpy="-1.5708 0 -1.5708"/>
-      <geometry>
-        <mesh filename="package://robot_description/meshes/joining_plate_t.stl"/>
-      </geometry>
-    </collision>
-    <!-- Part joining_plate_90_degree -->
-    <visual>
-      <origin xyz="0.180533 -1.01292 1.40652" rpy="-1.5708 -0 1.5708"/>
-      <geometry>
-        <mesh filename="package://robot_description/meshes/joining_plate_90_degree.stl"/>
+        <color rgba="0.866667 0.909804 1 1" />
+      </material>
+    </visual>
+    <collision>
+      <origin xyz="0.176533 -2.50295 1.40652" rpy="-1.5708 0 -1.5708" />
+      <geometry>
+        <mesh filename="./assets/joining_plate_t.stl" />
+      </geometry>
+    </collision>
+  </link>
+  <!-- Part joining_plate_90_degree -->
+  <link name="joining_plate_90_degree">
+    <visual>
+      <origin xyz="0.180533 -1.01292 1.40652" rpy="-1.5708 -0 1.5708" />
+      <geometry>
+        <mesh filename="./assets/joining_plate_90_degree.stl" />
       </geometry>
       <material name="joining_plate_90_degree_material">
-        <color rgba="0.866667 0.909804 1 1"/>
-      </material>
-    </visual>
-    <collision>
-      <origin xyz="0.180533 -1.01292 1.40652" rpy="-1.5708 -0 1.5708"/>
-      <geometry>
-        <mesh filename="package://robot_description/meshes/joining_plate_90_degree.stl"/>
-      </geometry>
-    </collision>
-    <!-- Part joining_plate_90_degree_2 -->
-    <visual>
-      <origin xyz="0.176533 -3.99292 1.40652" rpy="-1.5708 -0 -1.5708"/>
-      <geometry>
-        <mesh filename="package://robot_description/meshes/joining_plate_90_degree.stl"/>
+        <color rgba="0.866667 0.909804 1 1" />
+      </material>
+    </visual>
+    <collision>
+      <origin xyz="0.180533 -1.01292 1.40652" rpy="-1.5708 -0 1.5708" />
+      <geometry>
+        <mesh filename="./assets/joining_plate_90_degree.stl" />
+      </geometry>
+    </collision>
+  </link>
+  <!-- Part joining_plate_90_degree_2 -->
+  <link name="joining_plate_90_degree_2">
+    <visual>
+      <origin xyz="0.176533 -3.99292 1.40652" rpy="-1.5708 -0 -1.5708" />
+      <geometry>
+        <mesh filename="./assets/joining_plate_90_degree.stl" />
       </geometry>
       <material name="joining_plate_90_degree_2_material">
-        <color rgba="0.866667 0.909804 1 1"/>
-      </material>
-    </visual>
-    <collision>
-      <origin xyz="0.176533 -3.99292 1.40652" rpy="-1.5708 -0 -1.5708"/>
-      <geometry>
-        <mesh filename="package://robot_description/meshes/joining_plate_90_degree.stl"/>
-      </geometry>
-    </collision>
-    <!-- Part joining_plate_90_degree_3 -->
-    <visual>
-      <origin xyz="1.66153 -3.99292 1.40652" rpy="-1.5708 -0 -1.5708"/>
-      <geometry>
-        <mesh filename="package://robot_description/meshes/joining_plate_90_degree.stl"/>
+        <color rgba="0.866667 0.909804 1 1" />
+      </material>
+    </visual>
+    <collision>
+      <origin xyz="0.176533 -3.99292 1.40652" rpy="-1.5708 -0 -1.5708" />
+      <geometry>
+        <mesh filename="./assets/joining_plate_90_degree.stl" />
+      </geometry>
+    </collision>
+  </link>
+  <!-- Part joining_plate_90_degree_3 -->
+  <link name="joining_plate_90_degree_3">
+    <visual>
+      <origin xyz="1.66153 -3.99292 1.40652" rpy="-1.5708 -0 -1.5708" />
+      <geometry>
+        <mesh filename="./assets/joining_plate_90_degree.stl" />
       </geometry>
       <material name="joining_plate_90_degree_3_material">
-        <color rgba="0.866667 0.909804 1 1"/>
-      </material>
-    </visual>
-    <collision>
-      <origin xyz="1.66153 -3.99292 1.40652" rpy="-1.5708 -0 -1.5708"/>
-      <geometry>
-        <mesh filename="package://robot_description/meshes/joining_plate_90_degree.stl"/>
-      </geometry>
-    </collision>
-    <!-- Part joining_plate_90_degree_4 -->
-    <visual>
-      <origin xyz="1.68953 -1.01292 1.40652" rpy="-1.5708 -0 1.5708"/>
-      <geometry>
-        <mesh filename="package://robot_description/meshes/joining_plate_90_degree.stl"/>
+        <color rgba="0.866667 0.909804 1 1" />
+      </material>
+    </visual>
+    <collision>
+      <origin xyz="1.66153 -3.99292 1.40652" rpy="-1.5708 -0 -1.5708" />
+      <geometry>
+        <mesh filename="./assets/joining_plate_90_degree.stl" />
+      </geometry>
+    </collision>
+  </link>
+  <!-- Part joining_plate_90_degree_4 -->
+  <link name="joining_plate_90_degree_4">
+    <visual>
+      <origin xyz="1.68953 -1.01292 1.40652" rpy="-1.5708 -0 1.5708" />
+      <geometry>
+        <mesh filename="./assets/joining_plate_90_degree.stl" />
       </geometry>
       <material name="joining_plate_90_degree_4_material">
-        <color rgba="0.866667 0.909804 1 1"/>
-      </material>
-    </visual>
-    <collision>
-      <origin xyz="1.68953 -1.01292 1.40652" rpy="-1.5708 -0 1.5708"/>
-      <geometry>
-        <mesh filename="package://robot_description/meshes/joining_plate_90_degree.stl"/>
-      </geometry>
-    </collision>
-    <!-- Part joining_plate_90_degree_5 -->
-    <visual>
-      <origin xyz="1.66553 -1.01292 1.40652" rpy="-1.5708 -0 1.5708"/>
-      <geometry>
-        <mesh filename="package://robot_description/meshes/joining_plate_90_degree.stl"/>
+        <color rgba="0.866667 0.909804 1 1" />
+      </material>
+    </visual>
+    <collision>
+      <origin xyz="1.68953 -1.01292 1.40652" rpy="-1.5708 -0 1.5708" />
+      <geometry>
+        <mesh filename="./assets/joining_plate_90_degree.stl" />
+      </geometry>
+    </collision>
+  </link>
+  <!-- Part joining_plate_90_degree_5 -->
+  <link name="joining_plate_90_degree_5">
+    <visual>
+      <origin xyz="1.66553 -1.01292 1.40652" rpy="-1.5708 -0 1.5708" />
+      <geometry>
+        <mesh filename="./assets/joining_plate_90_degree.stl" />
       </geometry>
       <material name="joining_plate_90_degree_5_material">
-        <color rgba="0.866667 0.909804 1 1"/>
-      </material>
-    </visual>
-    <collision>
-      <origin xyz="1.66553 -1.01292 1.40652" rpy="-1.5708 -0 1.5708"/>
-      <geometry>
-        <mesh filename="package://robot_description/meshes/joining_plate_90_degree.stl"/>
-      </geometry>
-    </collision>
-    <!-- Part joining_plate_90_degree_6 -->
-    <visual>
-      <origin xyz="0.200533 -3.99292 1.40652" rpy="-1.5708 -0 -1.5708"/>
-      <geometry>
-        <mesh filename="package://robot_description/meshes/joining_plate_90_degree.stl"/>
+        <color rgba="0.866667 0.909804 1 1" />
+      </material>
+    </visual>
+    <collision>
+      <origin xyz="1.66553 -1.01292 1.40652" rpy="-1.5708 -0 1.5708" />
+      <geometry>
+        <mesh filename="./assets/joining_plate_90_degree.stl" />
+      </geometry>
+    </collision>
+  </link>
+  <!-- Part joining_plate_90_degree_6 -->
+  <link name="joining_plate_90_degree_6">
+    <visual>
+      <origin xyz="0.200533 -3.99292 1.40652" rpy="-1.5708 -0 -1.5708" />
+      <geometry>
+        <mesh filename="./assets/joining_plate_90_degree.stl" />
       </geometry>
       <material name="joining_plate_90_degree_6_material">
-        <color rgba="0.866667 0.909804 1 1"/>
-      </material>
-    </visual>
-    <collision>
-      <origin xyz="0.200533 -3.99292 1.40652" rpy="-1.5708 -0 -1.5708"/>
-      <geometry>
-        <mesh filename="package://robot_description/meshes/joining_plate_90_degree.stl"/>
-      </geometry>
-    </collision>
-    <!-- Part joining_plate_90_degree_7 -->
-    <visual>
-      <origin xyz="0.204533 -1.01292 1.40652" rpy="-1.5708 -0 1.5708"/>
-      <geometry>
-        <mesh filename="package://robot_description/meshes/joining_plate_90_degree.stl"/>
+        <color rgba="0.866667 0.909804 1 1" />
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