Commit message: fixed joints and package references. also fixed launch file after error

File: src/robot_description/urdf/robot.urdf.xacro (robot description, xacro)
@@ -17,5 +17,5 @@
       <origin xyz="1.67553 -2.50292 1.41602" rpy="0 -0 0" />
       <geometry>
-        <mesh filename="./assets/v_slot_20x40x1500_linear_rail.stl" />
+        <mesh filename="package://robot_description/meshes/v_slot_20x40x1500_linear_rail.stl" />
       </geometry>
       <material name="v_slot_20x40x1500_linear_rail_material">
@@ -26,5 +26,5 @@
       <origin xyz="1.67553 -2.50292 1.41602" rpy="0 -0 0" />
       <geometry>
-        <mesh filename="./assets/v_slot_20x40x1500_linear_rail.stl" />
+        <mesh filename="package://robot_description/meshes/v_slot_20x40x1500_linear_rail.stl" />
       </geometry>
     </collision>
@@ -35,5 +35,5 @@
       <origin xyz="0.190533 -1.00292 1.41602" rpy="0 -0 0" />
       <geometry>
-        <mesh filename="./assets/v_slot_20x40x1500_linear_rail.stl" />
+        <mesh filename="package://robot_description/meshes/v_slot_20x40x1500_linear_rail.stl" />
       </geometry>
       <material name="v_slot_20x40x1500_linear_rail_2_material">
@@ -44,5 +44,5 @@
       <origin xyz="0.190533 -1.00292 1.41602" rpy="0 -0 0" />
       <geometry>
-        <mesh filename="./assets/v_slot_20x40x1500_linear_rail.stl" />
+        <mesh filename="package://robot_description/meshes/v_slot_20x40x1500_linear_rail.stl" />
       </geometry>
     </collision>
@@ -53,5 +53,5 @@
       <origin xyz="0.190533 -2.50292 1.41602" rpy="0 -0 0" />
       <geometry>
-        <mesh filename="./assets/v_slot_20x40x1500_linear_rail.stl" />
+        <mesh filename="package://robot_description/meshes/v_slot_20x40x1500_linear_rail.stl" />
       </geometry>
       <material name="v_slot_20x40x1500_linear_rail_3_material">
@@ -62,5 +62,5 @@
       <origin xyz="0.190533 -2.50292 1.41602" rpy="0 -0 0" />
       <geometry>
-        <mesh filename="./assets/v_slot_20x40x1500_linear_rail.stl" />
+        <mesh filename="package://robot_description/meshes/v_slot_20x40x1500_linear_rail.stl" />
       </geometry>
     </collision>
@@ -71,5 +71,5 @@
       <origin xyz="1.67553 -1.00292 1.41602" rpy="0 -0 0" />
       <geometry>
-        <mesh filename="./assets/v_slot_20x40x1500_linear_rail.stl" />
+        <mesh filename="package://robot_description/meshes/v_slot_20x40x1500_linear_rail.stl" />
       </geometry>
       <material name="v_slot_20x40x1500_linear_rail_4_material">
@@ -80,5 +80,5 @@
       <origin xyz="1.67553 -1.00292 1.41602" rpy="0 -0 0" />
       <geometry>
-        <mesh filename="./assets/v_slot_20x40x1500_linear_rail.stl" />
+        <mesh filename="package://robot_description/meshes/v_slot_20x40x1500_linear_rail.stl" />
       </geometry>
     </collision>
@@ -89,5 +89,5 @@
       <origin xyz="1.68953 -2.50352 1.40652" rpy="-1.5708 -0 1.5708" />
       <geometry>
-        <mesh filename="./assets/joining_plate_t.stl" />
+        <mesh filename="package://robot_description/meshes/joining_plate_t.stl" />
       </geometry>
       <material name="joining_plate_t_material">
@@ -98,5 +98,5 @@
       <origin xyz="1.68953 -2.50352 1.40652" rpy="-1.5708 -0 1.5708" />
       <geometry>
-        <mesh filename="./assets/joining_plate_t.stl" />
+        <mesh filename="package://robot_description/meshes/joining_plate_t.stl" />
       </geometry>
     </collision>
@@ -107,5 +107,5 @@
       <origin xyz="0.176533 -2.50295 1.40652" rpy="-1.5708 0 -1.5708" />
       <geometry>
-        <mesh filename="./assets/joining_plate_t.stl" />
+        <mesh filename="package://robot_description/meshes/joining_plate_t.stl" />
       </geometry>
       <material name="joining_plate_t_2_material">
@@ -116,5 +116,5 @@
       <origin xyz="0.176533 -2.50295 1.40652" rpy="-1.5708 0 -1.5708" />
       <geometry>
-        <mesh filename="./assets/joining_plate_t.stl" />
+        <mesh filename="package://robot_description/meshes/joining_plate_t.stl" />
       </geometry>
     </collision>
@@ -125,5 +125,5 @@
       <origin xyz="0.180533 -1.01292 1.40652" rpy="-1.5708 -0 1.5708" />
       <geometry>
-        <mesh filename="./assets/joining_plate_90_degree.stl" />
+        <mesh filename="package://robot_description/meshes/joining_plate_90_degree.stl" />
       </geometry>
       <material name="joining_plate_90_degree_material">
@@ -134,5 +134,5 @@
       <origin xyz="0.180533 -1.01292 1.40652" rpy="-1.5708 -0 1.5708" />
       <geometry>
-        <mesh filename="./assets/joining_plate_90_degree.stl" />
+        <mesh filename="package://robot_description/meshes/joining_plate_90_degree.stl" />
       </geometry>
     </collision>
@@ -143,5 +143,5 @@
       <origin xyz="0.176533 -3.99292 1.40652" rpy="-1.5708 -0 -1.5708" />
       <geometry>
-        <mesh filename="./assets/joining_plate_90_degree.stl" />
+        <mesh filename="package://robot_description/meshes/joining_plate_90_degree.stl" />
       </geometry>
       <material name="joining_plate_90_degree_2_material">
@@ -152,5 +152,5 @@
       <origin xyz="0.176533 -3.99292 1.40652" rpy="-1.5708 -0 -1.5708" />
       <geometry>
-        <mesh filename="./assets/joining_plate_90_degree.stl" />
+        <mesh filename="package://robot_description/meshes/joining_plate_90_degree.stl" />
       </geometry>
     </collision>
@@ -161,5 +161,5 @@
       <origin xyz="1.66153 -3.99292 1.40652" rpy="-1.5708 -0 -1.5708" />
       <geometry>
-        <mesh filename="./assets/joining_plate_90_degree.stl" />
+        <mesh filename="package://robot_description/meshes/joining_plate_90_degree.stl" />
       </geometry>
       <material name="joining_plate_90_degree_3_material">
@@ -170,5 +170,5 @@
       <origin xyz="1.66153 -3.99292 1.40652" rpy="-1.5708 -0 -1.5708" />
       <geometry>
-        <mesh filename="./assets/joining_plate_90_degree.stl" />
+        <mesh filename="package://robot_description/meshes/joining_plate_90_degree.stl" />
       </geometry>
     </collision>
@@ -179,5 +179,5 @@
       <origin xyz="1.68953 -1.01292 1.40652" rpy="-1.5708 -0 1.5708" />
       <geometry>
-        <mesh filename="./assets/joining_plate_90_degree.stl" />
+        <mesh filename="package://robot_description/meshes/joining_plate_90_degree.stl" />
       </geometry>
       <material name="joining_plate_90_degree_4_material">
@@ -188,5 +188,5 @@
       <origin xyz="1.68953 -1.01292 1.40652" rpy="-1.5708 -0 1.5708" />
       <geometry>
-        <mesh filename="./assets/joining_plate_90_degree.stl" />
+        <mesh filename="package://robot_description/meshes/joining_plate_90_degree.stl" />
       </geometry>
     </collision>
@@ -197,5 +197,5 @@
       <origin xyz="1.66553 -1.01292 1.40652" rpy="-1.5708 -0 1.5708" />
       <geometry>
-        <mesh filename="./assets/joining_plate_90_degree.stl" />
+        <mesh filename="package://robot_description/meshes/joining_plate_90_degree.stl" />
       </geometry>
       <material name="joining_plate_90_degree_5_material">
@@ -206,5 +206,5 @@
       <origin xyz="1.66553 -1.01292 1.40652" rpy="-1.5708 -0 1.5708" />
       <geometry>
-        <mesh filename="./assets/joining_plate_90_degree.stl" />
+        <mesh filename="package://robot_description/meshes/joining_plate_90_degree.stl" />
       </geometry>
     </collision>
@@ -215,5 +215,5 @@
       <origin xyz="0.200533 -3.99292 1.40652" rpy="-1.5708 -0 -1.5708" />
       <geometry>
-        <mesh filename="./assets/joining_plate_90_degree.stl" />
+        <mesh filename="package://robot_description/meshes/joining_plate_90_degree.stl" />
       </geometry>
       <material name="joining_plate_90_degree_6_material">
@@ -224,5 +224,5 @@
       <origin xyz="0.200533 -3.99292 1.40652" rpy="-1.5708 -0 -1.5708" />
       <geometry>
-        <mesh filename="./assets/joining_plate_90_degree.stl" />
+        <mesh filename="package://robot_description/meshes/joining_plate_90_degree.stl" />
       </geometry>
     </collision>
@@ -233,5 +233,5 @@
       <origin xyz="0.204533 -1.01292 1.40652" rpy="-1.5708 -0 1.5708" />
       <geometry>
-        <mesh filename="./assets/joining_plate_90_degree.stl" />
+        <mesh filename="package://robot_description/meshes/joining_plate_90_degree.stl" />
       </geometry>
       <material name="joining_plate_90_degree_7_material">
@@ -242,5 +242,5 @@
       <origin xyz="0.204533 -1.01292 1.40652" rpy="-1.5708 -0 1.5708" />
       <geometry>
-        <mesh filename="./assets/joining_plate_90_degree.stl" />
+        <mesh filename="package://robot_description/meshes/joining_plate_90_degree.stl" />
       </geometry>
     </collision>
@@ -251,5 +251,5 @@
       <origin xyz="1.68553 -3.99292 1.40652" rpy="-1.5708 -0 -1.5708" />
       <geometry>
-        <mesh filename="./assets/joining_plate_90_degree.stl" />
+        <mesh filename="package://robot_description/meshes/joining_plate_90_degree.stl" />
       </geometry>
       <material name="joining_plate_90_degree_8_material">
@@ -260,5 +260,5 @@
       <origin xyz="1.68553 -3.99292 1.40652" rpy="-1.5708 -0 -1.5708" />
       <geometry>
-        <mesh filename="./assets/joining_plate_90_degree.stl" />
+        <mesh filename="package://robot_description/meshes/joining_plate_90_degree.stl" />
       </geometry>
     </collision>
@@ -269,5 +269,5 @@
       <origin xyz="1.67381 -2.02484 3.19503" rpy="1.5708 -1.5708 0" />
       <geometry>
-        <mesh filename="./assets/joining_plate_90_degree.stl" />
+        <mesh filename="package://robot_description/meshes/joining_plate_90_degree.stl" />
       </geometry>
       <material name="joining_plate_90_degree_9_material">
@@ -278,5 +278,5 @@
       <origin xyz="1.67381 -2.02484 3.19503" rpy="1.5708 -1.5708 0" />
       <geometry>
-        <mesh filename="./assets/joining_plate_90_degree.stl" />
+        <mesh filename="package://robot_description/meshes/joining_plate_90_degree.stl" />
       </geometry>
     </collision>
@@ -287,5 +287,5 @@
       <origin xyz="0.19385 -2.06955 3.18355" rpy="1.5708 -0 -3.14159" />
       <geometry>
-        <mesh filename="./assets/v_slot_20x80x200_linear_rail.stl" />
+        <mesh filename="package://robot_description/meshes/v_slot_20x80x200_linear_rail.stl" />
       </geometry>
       <material name="v_slot_20x80x200_linear_rail_material">
@@ -296,5 +296,5 @@
       <origin xyz="0.19385 -2.06955 3.18355" rpy="1.5708 -0 -3.14159" />
       <geometry>
-        <mesh filename="./assets/v_slot_20x80x200_linear_rail.stl" />
+        <mesh filename="package://robot_description/meshes/v_slot_20x80x200_linear_rail.stl" />
       </geometry>
     </collision>
@@ -305,5 +305,5 @@
       <origin xyz="0.20475 -2.06905 1.53655" rpy="-0 0 -1.5708" />
       <geometry>
-        <mesh filename="./assets/gantry_column_base_plate.stl" />
+        <mesh filename="package://robot_description/meshes/gantry_column_base_plate.stl" />
       </geometry>
       <material name="gantry_column_base_plate_material">
@@ -314,5 +314,5 @@
       <origin xyz="0.20475 -2.06905 1.53655" rpy="-0 0 -1.5708" />
       <geometry>
-        <mesh filename="./assets/gantry_column_base_plate.stl" />
+        <mesh filename="package://robot_description/meshes/gantry_column_base_plate.stl" />
       </geometry>
     </collision>
@@ -323,5 +323,5 @@
       <origin xyz="0.19385 -2.06955 2.98355" rpy="1.5708 -0 -3.14159" />
       <geometry>
-        <mesh filename="./assets/v_slot_20x80x1500_linear_rail.stl" />
+        <mesh filename="package://robot_description/meshes/v_slot_20x80x1500_linear_rail.stl" />
       </geometry>
       <material name="v_slot_20x80x1500_linear_rail_material">
@@ -332,5 +332,5 @@
       <origin xyz="0.19385 -2.06955 2.98355" rpy="1.5708 -0 -3.14159" />
       <geometry>
-        <mesh filename="./assets/v_slot_20x80x1500_linear_rail.stl" />
+        <mesh filename="package://robot_description/meshes/v_slot_20x80x1500_linear_rail.stl" />
       </geometry>
     </collision>
@@ -341,5 +341,5 @@
       <origin xyz="0.19435 -2.02955 3.19534" rpy="-1.5708 -1.5708 0" />
       <geometry>
-        <mesh filename="./assets/joining_plate_90_degree.stl" />
+        <mesh filename="package://robot_description/meshes/joining_plate_90_degree.stl" />
       </geometry>
       <material name="joining_plate_90_degree_10_material">
@@ -350,5 +350,5 @@
       <origin xyz="0.19435 -2.02955 3.19534" rpy="-1.5708 -1.5708 0" />
       <geometry>
-        <mesh filename="./assets/joining_plate_90_degree.stl" />
+        <mesh filename="package://robot_description/meshes/joining_plate_90_degree.stl" />
       </geometry>
     </collision>
@@ -359,5 +359,5 @@
       <origin xyz="1.67381 -2.10884 3.1952" rpy="1.5708 -1.5708 0" />
       <geometry>
-        <mesh filename="./assets/joining_plate_90_degree.stl" />
+        <mesh filename="package://robot_description/meshes/joining_plate_90_degree.stl" />
       </geometry>
       <material name="joining_plate_90_degree_11_material">
@@ -368,5 +368,5 @@
       <origin xyz="1.67381 -2.10884 3.1952" rpy="1.5708 -1.5708 0" />
       <geometry>
-        <mesh filename="./assets/joining_plate_90_degree.stl" />
+        <mesh filename="package://robot_description/meshes/joining_plate_90_degree.stl" />
       </geometry>
     </collision>
@@ -377,5 +377,5 @@
       <origin xyz="0.19435 -2.10955 3.19305" rpy="-1.5708 -0 -3.14159" />
       <geometry>
-        <mesh filename="./assets/joining_plate_90_degree.stl" />
+        <mesh filename="package://robot_description/meshes/joining_plate_90_degree.stl" />
       </geometry>
       <material name="joining_plate_90_degree_12_material">
@@ -386,5 +386,5 @@
       <origin xyz="0.19435 -2.10955 3.19305" rpy="-1.5708 -0 -3.14159" />
       <geometry>
-        <mesh filename="./assets/joining_plate_90_degree.stl" />
+        <mesh filename="package://robot_description/meshes/joining_plate_90_degree.stl" />
       </geometry>
     </collision>
@@ -395,5 +395,5 @@
       <origin xyz="0.18385 -2.03955 3.20355" rpy="0 -0 1.5708" />
       <geometry>
-        <mesh filename="./assets/v_slot_20x40x1500_linear_rail.stl" />
+        <mesh filename="package://robot_description/meshes/v_slot_20x40x1500_linear_rail.stl" />
       </geometry>
       <material name="v_slot_20x40x1500_linear_rail_5_material">
@@ -404,5 +404,5 @@
       <origin xyz="0.18385 -2.03955 3.20355" rpy="0 -0 1.5708" />
       <geometry>
-        <mesh filename="./assets/v_slot_20x40x1500_linear_rail.stl" />
+        <mesh filename="package://robot_description/meshes/v_slot_20x40x1500_linear_rail.stl" />
       </geometry>
     </collision>
@@ -413,5 +413,5 @@
       <origin xyz="0.18385 -2.09955 3.20355" rpy="0 -0 1.5708" />
       <geometry>
-        <mesh filename="./assets/v_slot_20x40x1500_linear_rail.stl" />
+        <mesh filename="package://robot_description/meshes/v_slot_20x40x1500_linear_rail.stl" />
       </geometry>
       <material name="v_slot_20x40x1500_linear_rail_6_material">
@@ -422,5 +422,5 @@
       <origin xyz="0.18385 -2.09955 3.20355" rpy="0 -0 1.5708" />
       <geometry>
-        <mesh filename="./assets/v_slot_20x40x1500_linear_rail.stl" />
+        <mesh filename="package://robot_description/meshes/v_slot_20x40x1500_linear_rail.stl" />
       </geometry>
     </collision>
@@ -431,5 +431,5 @@
       <origin xyz="1.67431 -2.06884 3.18355" rpy="1.5708 -0 0" />
       <geometry>
-        <mesh filename="./assets/v_slot_20x80x200_linear_rail.stl" />
+        <mesh filename="package://robot_description/meshes/v_slot_20x80x200_linear_rail.stl" />
       </geometry>
       <material name="v_slot_20x80x200_linear_rail_2_material">
@@ -440,5 +440,5 @@
       <origin xyz="1.67431 -2.06884 3.18355" rpy="1.5708 -0 0" />
       <geometry>
-        <mesh filename="./assets/v_slot_20x80x200_linear_rail.stl" />
+        <mesh filename="package://robot_description/meshes/v_slot_20x80x200_linear_rail.stl" />
       </geometry>
     </collision>
@@ -449,5 +449,5 @@
       <origin xyz="1.66341 -2.06934 1.53655" rpy="-0 0 1.5708" />
       <geometry>
-        <mesh filename="./assets/gantry_column_base_plate.stl" />
+        <mesh filename="package://robot_description/meshes/gantry_column_base_plate.stl" />
       </geometry>
       <material name="gantry_column_base_plate_2_material">
@@ -458,5 +458,5 @@
       <origin xyz="1.66341 -2.06934 1.53655" rpy="-0 0 1.5708" />
       <geometry>
-        <mesh filename="./assets/gantry_column_base_plate.stl" />
+        <mesh filename="package://robot_description/meshes/gantry_column_base_plate.stl" />
       </geometry>
     </collision>
@@ -467,5 +467,5 @@
       <origin xyz="1.67431 -2.06884 2.98355" rpy="1.5708 -0 0" />
       <geometry>
-        <mesh filename="./assets/v_slot_20x80x1500_linear_rail.stl" />
+        <mesh filename="package://robot_description/meshes/v_slot_20x80x1500_linear_rail.stl" />
       </geometry>
       <material name="v_slot_20x80x1500_linear_rail_2_material">
@@ -476,5 +476,5 @@
       <origin xyz="1.67431 -2.06884 2.98355" rpy="1.5708 -0 0" />
       <geometry>
-        <mesh filename="./assets/v_slot_20x80x1500_linear_rail.stl" />
+        <mesh filename="package://robot_description/meshes/v_slot_20x80x1500_linear_rail.stl" />
       </geometry>
     </collision>
@@ -485,5 +485,5 @@
       <origin xyz="1.68023 -2.50352 1.40652" rpy="-1.5708 1.5708 0" />
       <geometry>
-        <mesh filename="./assets/m5_tee_nut.stl" />
+        <mesh filename="package://robot_description/meshes/m5_tee_nut.stl" />
       </geometry>
       <material name="m5_tee_nut_material">
@@ -494,5 +494,5 @@
       <origin xyz="1.68023 -2.50352 1.40652" rpy="-1.5708 1.5708 0" />
       <geometry>
-        <mesh filename="./assets/m5_tee_nut.stl" />
+        <mesh filename="package://robot_description/meshes/m5_tee_nut.stl" />
       </geometry>
     </collision>
@@ -503,5 +503,5 @@
       <origin xyz="1.68953 -2.50352 1.40652" rpy="-1.5708 1.5708 0" />
       <geometry>
-        <mesh filename="./assets/m5_x_10mm_screw.stl" />
+        <mesh filename="package://robot_description/meshes/m5_x_10mm_screw.stl" />
       </geometry>
       <material name="m5_x_10mm_screw_material">
@@ -512,5 +512,5 @@
       <origin xyz="1.68953 -2.50352 1.40652" rpy="-1.5708 1.5708 0" />
       <geometry>
-        <mesh filename="./assets/m5_x_10mm_screw.stl" />
+        <mesh filename="package://robot_description/meshes/m5_x_10mm_screw.stl" />
       </geometry>
     </collision>
@@ -521,5 +521,5 @@
       <origin xyz="1.68023 -2.48352 1.40652" rpy="-1.5708 1.5708 0" />
       <geometry>
-        <mesh filename="./assets/m5_tee_nut.stl" />
+        <mesh filename="package://robot_description/meshes/m5_tee_nut.stl" />
       </geometry>
       <material name="m5_tee_nut_2_material">
@@ -530,5 +530,5 @@
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
Commit message: robot fixes

File: src/robot_description/urdf/robot.urdf.xacro (robot description, xacro)
@@ -4,4 +4,11 @@
 https://cad.onshape.com/documents/a2e4d90d4720e7eb81b47647/w/f29fb00f1617a93c8228a45a/e/cddef7938b795a6053ad7145 -->
 <robot name="surgeyos-robot2">
+  <!-- Global placement: center robot in XY at the world origin while keeping floor at z=0. -->
+  <link name="world" />
+  <joint name="world_to_robot" type="fixed">
+    <parent link="world" />
+    <child link="x_axis_tracks_inertial" />
+    <origin xyz="-0.898235 1.99646 -1.35" rpy="0 0 0" />
+  </joint>
   <!-- Link x_axis_tracks -->
   <link name="x_axis_tracks_inertial">
