Commit message: updated robot

File: src/robot_description/urdf/robot.urdf.xacro (robot description, xacro)
@@ -1,12509 +1,5693 @@
-<?xml version="1.0"?>
+<?xml version="1.0" ?>
 <!-- Generated using onshape-to-robot -->
-<!-- Onshape
-https://cad.onshape.com/documents/a2e4d90d4720e7eb81b47647/w/f29fb00f1617a93c8228a45a/e/cddef7938b795a6053ad7145 -->
-<robot name="surgeyos-robot2">
-  <!-- Global placement: center robot in XY at the world origin while keeping floor at z=0. -->
-  <link name="world" />
-  <joint name="world_to_robot" type="fixed">
-    <parent link="world" />
-    <child link="x_axis_tracks_inertial" />
-    <origin xyz="-0.898235 1.99646 -1.35" rpy="0 0 0" />
+<!-- Onshape https://cad.onshape.com/documents/a2e4d90d4720e7eb81b47647/w/f29fb00f1617a93c8228a45a/e/5adbd4e56813ca0b03de2f98 -->
+<robot name="onshape-to-robot">
+  <!-- Link body -->
+  <link name="body">
+    <inertial>
+      <origin xyz="0 0 0" rpy="0 0 0"/>
+      <mass value="1e-09"/>
+      <inertia ixx="1e-09" ixy="0" ixz="0" iyy="1e-09" iyz="0" izz="1e-09"/>
+    </inertial>
+    <!-- Part v_slot_20x40x1500_linear_rail -->
+    <visual>
+      <origin xyz="1.03456 -1.44349 0.368183" rpy="-0 -0 0.011542"/>
+      <geometry>
+        <mesh filename="package://robot_description/assets/v_slot_20x40x1500_linear_rail.stl"/>
+      </geometry>
+      <material name="v_slot_20x40x1500_linear_rail_material">
+        <color rgba="0.866667 0.909804 1 1"/>
+      </material>
+    </visual>
+    <collision>
+      <origin xyz="1.03456 -1.44349 0.368183" rpy="-0 -0 0.011542"/>
+      <geometry>
+        <mesh filename="package://robot_description/assets/v_slot_20x40x1500_linear_rail.stl"/>
+      </geometry>
+    </collision>
+    <!-- Part v_slot_20x40x1500_linear_rail_2 -->
+    <visual>
+      <origin xyz="-0.45034 -1.46063 0.368183" rpy="-0 -0 0.011542"/>
+      <geometry>
+        <mesh filename="package://robot_description/assets/v_slot_20x40x1500_linear_rail.stl"/>
+      </geometry>
+      <material name="v_slot_20x40x1500_linear_rail_2_material">
+        <color rgba="0.866667 0.909804 1 1"/>
+      </material>
+    </visual>
+    <collision>
+      <origin xyz="-0.45034 -1.46063 0.368183" rpy="-0 -0 0.011542"/>
+      <geometry>
+        <mesh filename="package://robot_description/assets/v_slot_20x40x1500_linear_rail.stl"/>
+      </geometry>
+    </collision>
+    <!-- Part v_slot_20x40x1500_linear_rail_3 -->
+    <visual>
+      <origin xyz="-0.467653 0.0392729 0.368183" rpy="-0 -0 0.011542"/>
+      <geometry>
+        <mesh filename="package://robot_description/assets/v_slot_20x40x1500_linear_rail.stl"/>
+      </geometry>
+      <material name="v_slot_20x40x1500_linear_rail_3_material">
+        <color rgba="0.866667 0.909804 1 1"/>
+      </material>
+    </visual>
+    <collision>
+      <origin xyz="-0.467653 0.0392729 0.368183" rpy="-0 -0 0.011542"/>
+      <geometry>
+        <mesh filename="package://robot_description/assets/v_slot_20x40x1500_linear_rail.stl"/>
+      </geometry>
+    </collision>
+    <!-- Part v_slot_20x40x1500_linear_rail_4 -->
+    <visual>
+      <origin xyz="1.01725 0.0564124 0.368183" rpy="-0 -0 0.011542"/>
+      <geometry>
+        <mesh filename="package://robot_description/assets/v_slot_20x40x1500_linear_rail.stl"/>
+      </geometry>
+      <material name="v_slot_20x40x1500_linear_rail_4_material">
+        <color rgba="0.866667 0.909804 1 1"/>
+      </material>
+    </visual>
+    <collision>
+      <origin xyz="1.01725 0.0564124 0.368183" rpy="-0 -0 0.011542"/>
+      <geometry>
+        <mesh filename="package://robot_description/assets/v_slot_20x40x1500_linear_rail.stl"/>
+      </geometry>
+    </collision>
+    <!-- Part joining_plate_t -->
+    <visual>
+      <origin xyz="1.04857 -1.44393 0.358683" rpy="-1.5708 0 1.58234"/>
+      <geometry>
+        <mesh filename="package://robot_description/assets/joining_plate_t.stl"/>
+      </geometry>
+      <material name="joining_plate_t_material">
+        <color rgba="0.866667 0.909804 1 1"/>
+      </material>
+    </visual>
+    <collision>
+      <origin xyz="1.04857 -1.44393 0.358683" rpy="-1.5708 0 1.58234"/>
+      <geometry>
+        <mesh filename="package://robot_description/assets/joining_plate_t.stl"/>
+      </geometry>
+    </collision>
+    <!-- Part joining_plate_t_2 -->
+    <visual>
+      <origin xyz="-0.464339 -1.46082 0.358683" rpy="-1.5708 -0 -1.55925"/>
+      <geometry>
+        <mesh filename="package://robot_description/assets/joining_plate_t.stl"/>
+      </geometry>
+      <material name="joining_plate_t_2_material">
+        <color rgba="0.866667 0.909804 1 1"/>
+      </material>
+    </visual>
+    <collision>
+      <origin xyz="-0.464339 -1.46082 0.358683" rpy="-1.5708 -0 -1.55925"/>
+      <geometry>
+        <mesh filename="package://robot_description/assets/joining_plate_t.stl"/>
+      </geometry>
+    </collision>
+    <!-- Part joining_plate_90_degree -->
+    <visual>
+      <origin xyz="-0.477537 0.0291582 0.358683" rpy="-1.5708 0 1.58234"/>
+      <geometry>
+        <mesh filename="package://robot_description/assets/joining_plate_90_degree.stl"/>
+      </geometry>
+      <material name="joining_plate_90_degree_material">
+        <color rgba="0.866667 0.909804 1 1"/>
+      </material>
+    </visual>
+    <collision>
+      <origin xyz="-0.477537 0.0291582 0.358683" rpy="-1.5708 0 1.58234"/>
+      <geometry>
+        <mesh filename="package://robot_description/assets/joining_plate_90_degree.stl"/>
+      </geometry>
+    </collision>
+    <!-- Part joining_plate_90_degree_2 -->
+    <visual>
+      <origin xyz="-0.447142 -2.95069 0.358683" rpy="-1.5708 -0 -1.55925"/>
+      <geometry>
+        <mesh filename="package://robot_description/assets/joining_plate_90_degree.stl"/>
+      </geometry>
+      <material name="joining_plate_90_degree_2_material">
+        <color rgba="0.866667 0.909804 1 1"/>
+      </material>
+    </visual>
+    <collision>
+      <origin xyz="-0.447142 -2.95069 0.358683" rpy="-1.5708 -0 -1.55925"/>
+      <geometry>
+        <mesh filename="package://robot_description/assets/joining_plate_90_degree.stl"/>
+      </geometry>
+    </collision>
+    <!-- Part joining_plate_90_degree_3 -->
+    <visual>
+      <origin xyz="1.03776 -2.93355 0.358683" rpy="-1.5708 -0 -1.55925"/>
+      <geometry>
+        <mesh filename="package://robot_description/assets/joining_plate_90_degree.stl"/>
+      </geometry>
+      <material name="joining_plate_90_degree_3_material">
+        <color rgba="0.866667 0.909804 1 1"/>
+      </material>
+    </visual>
+    <collision>
+      <origin xyz="1.03776 -2.93355 0.358683" rpy="-1.5708 -0 -1.55925"/>
+      <geometry>
+        <mesh filename="package://robot_description/assets/joining_plate_90_degree.stl"/>
+      </geometry>
+    </collision>
+    <!-- Part joining_plate_90_degree_4 -->
+    <visual>
+      <origin xyz="1.03136 0.0465746 0.358683" rpy="-1.5708 0 1.58234"/>
+      <geometry>
+        <mesh filename="package://robot_description/assets/joining_plate_90_degree.stl"/>
+      </geometry>
+      <material name="joining_plate_90_degree_4_material">
+        <color rgba="0.866667 0.909804 1 1"/>
+      </material>
+    </visual>
+    <collision>
+      <origin xyz="1.03136 0.0465746 0.358683" rpy="-1.5708 0 1.58234"/>
+      <geometry>
+        <mesh filename="package://robot_description/assets/joining_plate_90_degree.stl"/>
+      </geometry>
+    </collision>
+    <!-- Part joining_plate_90_degree_5 -->
+    <visual>
+      <origin xyz="1.00736 0.0462976 0.358683" rpy="-1.5708 0 1.58234"/>
+      <geometry>
+        <mesh filename="package://robot_description/assets/joining_plate_90_degree.stl"/>
+      </geometry>
+      <material name="joining_plate_90_degree_5_material">
+        <color rgba="0.866667 0.909804 1 1"/>
+      </material>
+    </visual>
+    <collision>
+      <origin xyz="1.00736 0.0462976 0.358683" rpy="-1.5708 0 1.58234"/>
+      <geometry>
+        <mesh filename="package://robot_description/assets/joining_plate_90_degree.stl"/>
+      </geometry>
+    </collision>
+    <!-- Part joining_plate_90_degree_6 -->
+    <visual>
+      <origin xyz="-0.423144 -2.95041 0.358683" rpy="-1.5708 -0 -1.55925"/>
+      <geometry>
+        <mesh filename="package://robot_description/assets/joining_plate_90_degree.stl"/>
+      </geometry>
+      <material name="joining_plate_90_degree_6_material">
+        <color rgba="0.866667 0.909804 1 1"/>
+      </material>
+    </visual>
+    <collision>
+      <origin xyz="-0.423144 -2.95041 0.358683" rpy="-1.5708 -0 -1.55925"/>
+      <geometry>
+        <mesh filename="package://robot_description/assets/joining_plate_90_degree.stl"/>
+      </geometry>
+    </collision>
+    <!-- Part joining_plate_90_degree_7 -->
+    <visual>
+      <origin xyz="-0.453539 0.0294352 0.358683" rpy="-1.5708 0 1.58234"/>
+      <geometry>
+        <mesh filename="package://robot_description/assets/joining_plate_90_degree.stl"/>
+      </geometry>
+      <material name="joining_plate_90_degree_7_material">
+        <color rgba="0.866667 0.909804 1 1"/>
+      </material>
+    </visual>
+    <collision>
+      <origin xyz="-0.453539 0.0294352 0.358683" rpy="-1.5708 0 1.58234"/>
+      <geometry>
+        <mesh filename="package://robot_description/assets/joining_plate_90_degree.stl"/>
+      </geometry>
+    </collision>
+    <!-- Part joining_plate_90_degree_8 -->
+    <visual>
+      <origin xyz="1.06176 -2.93327 0.358683" rpy="-1.5708 -0 -1.55925"/>
+      <geometry>
+        <mesh filename="package://robot_description/assets/joining_plate_90_degree.stl"/>
+      </geometry>
+      <material name="joining_plate_90_degree_8_material">
+        <color rgba="0.866667 0.909804 1 1"/>
+      </material>
+    </visual>
+    <collision>
+      <origin xyz="1.06176 -2.93327 0.358683" rpy="-1.5708 -0 -1.55925"/>
+      <geometry>
+        <mesh filename="package://robot_description/assets/joining_plate_90_degree.stl"/>
+      </geometry>
+    </collision>
+    <!-- Part m5_tee_nut -->
+    <visual>
+      <origin xyz="1.03927 -1.44403 0.358683" rpy="-1.58234 1.5708 0"/>
+      <geometry>
+        <mesh filename="package://robot_description/assets/m5_tee_nut.stl"/>
+      </geometry>
+      <material name="m5_tee_nut_material">
+        <color rgba="0.792157 0.819608 0.933333 1"/>
+      </material>
+    </visual>
+    <collision>
+      <origin xyz="1.03927 -1.44403 0.358683" rpy="-1.58234 1.5708 0"/>
+      <geometry>
+        <mesh filename="package://robot_description/assets/m5_tee_nut.stl"/>
+      </geometry>
+    </collision>
+    <!-- Part m5_x_10mm_screw -->
+    <visual>
+      <origin xyz="1.04857 -1.44393 0.358683" rpy="-1.58234 1.5708 0"/>
+      <geometry>
+        <mesh filename="package://robot_description/assets/m5_x_10mm_screw.stl"/>
+      </geometry>
+      <material name="m5_x_10mm_screw_material">
+        <color rgba="0.945098 0.94902 0.952941 1"/>
+      </material>
+    </visual>
+    <collision>
+      <origin xyz="1.04857 -1.44393 0.358683" rpy="-1.58234 1.5708 0"/>
+      <geometry>
+        <mesh filename="package://robot_description/assets/m5_x_10mm_screw.stl"/>
+      </geometry>
+    </collision>
+    <!-- Part m5_tee_nut_2 -->
+    <visual>
+      <origin xyz="1.03904 -1.42403 0.358683" rpy="-1.58234 1.5708 0"/>
+      <geometry>
+        <mesh filename="package://robot_description/assets/m5_tee_nut.stl"/>
+      </geometry>
+      <material name="m5_tee_nut_2_material">
+        <color rgba="0.792157 0.819608 0.933333 1"/>
+      </material>
+    </visual>
+    <collision>
+      <origin xyz="1.03904 -1.42403 0.358683" rpy="-1.58234 1.5708 0"/>
+      <geometry>
+        <mesh filename="package://robot_description/assets/m5_tee_nut.stl"/>
+      </geometry>
+    </collision>
+    <!-- Part m5_x_10mm_screw_2 -->
+    <visual>
+      <origin xyz="1.04834 -1.42393 0.358683" rpy="-1.58234 1.5708 0"/>
+      <geometry>
+        <mesh filename="package://robot_description/assets/m5_x_10mm_screw.stl"/>
+      </geometry>
+      <material name="m5_x_10mm_screw_2_material">
+        <color rgba="0.945098 0.94902 0.952941 1"/>
+      </material>
+    </visual>
+    <collision>
+      <origin xyz="1.04834 -1.42393 0.358683" rpy="-1.58234 1.5708 0"/>
+      <geometry>
+        <mesh filename="package://robot_description/assets/m5_x_10mm_screw.stl"/>
+      </geometry>
+    </collision>
+    <!-- Part m5_tee_nut_3 -->
+    <visual>
+      <origin xyz="1.0395 -1.46403 0.358683" rpy="-1.58234 1.5708 0"/>
+      <geometry>
+        <mesh filename="package://robot_description/assets/m5_tee_nut.stl"/>
+      </geometry>
+      <material name="m5_tee_nut_3_material">
+        <color rgba="0.792157 0.819608 0.933333 1"/>
+      </material>
+    </visual>
+    <collision>
+      <origin xyz="1.0395 -1.46403 0.358683" rpy="-1.58234 1.5708 0"/>
+      <geometry>
+        <mesh filename="package://robot_description/assets/m5_tee_nut.stl"/>
+      </geometry>
+    </collision>
+    <!-- Part m5_x_10mm_screw_3 -->
+    <visual>
+      <origin xyz="1.0488 -1.46392 0.358683" rpy="-1.58234 1.5708 0"/>
+      <geometry>
+        <mesh filename="package://robot_description/assets/m5_x_10mm_screw.stl"/>
+      </geometry>
+      <material name="m5_x_10mm_screw_3_material">
+        <color rgba="0.945098 0.94902 0.952941 1"/>
+      </material>
+    </visual>
+    <collision>
+      <origin xyz="1.0488 -1.46392 0.358683" rpy="-1.58234 1.5708 0"/>
+      <geometry>
+        <mesh filename="package://robot_description/assets/m5_x_10mm_screw.stl"/>
+      </geometry>
+    </collision>
+    <!-- Part m5_tee_nut_4 -->
+    <visual>
+      <origin xyz="-0.45504 -1.46071 0.358683" rpy="1.55925 1.5708 0"/>
+      <geometry>
+        <mesh filename="package://robot_description/assets/m5_tee_nut.stl"/>
+      </geometry>
+      <material name="m5_tee_nut_4_material">
+        <color rgba="0.792157 0.819608 0.933333 1"/>
+      </material>
+    </visual>
+    <collision>
+      <origin xyz="-0.45504 -1.46071 0.358683" rpy="1.55925 1.5708 0"/>
+      <geometry>
+        <mesh filename="package://robot_description/assets/m5_tee_nut.stl"/>
+      </geometry>
+    </collision>
+    <!-- Part m5_x_10mm_screw_4 -->
+    <visual>
+      <origin xyz="-0.464339 -1.46082 0.358683" rpy="1.55925 1.5708 0"/>
+      <geometry>
+        <mesh filename="package://robot_description/assets/m5_x_10mm_screw.stl"/>
+      </geometry>
+      <material name="m5_x_10mm_screw_4_material">
+        <color rgba="0.945098 0.94902 0.952941 1"/>
+      </material>
+    </visual>
+    <collision>
+      <origin xyz="-0.464339 -1.46082 0.358683" rpy="1.55925 1.5708 0"/>
+      <geometry>
+        <mesh filename="package://robot_description/assets/m5_x_10mm_screw.stl"/>
+      </geometry>
+    </collision>
+    <!-- Part m5_tee_nut_5 -->
+    <visual>
+      <origin xyz="-0.454809 -1.48071 0.358683" rpy="1.55925 1.5708 0"/>
+      <geometry>
+        <mesh filename="package://robot_description/assets/m5_tee_nut.stl"/>
+      </geometry>
+      <material name="m5_tee_nut_5_material">
+        <color rgba="0.792157 0.819608 0.933333 1"/>
+      </material>
+    </visual>
+    <collision>
+      <origin xyz="-0.454809 -1.48071 0.358683" rpy="1.55925 1.5708 0"/>
+      <geometry>
+        <mesh filename="package://robot_description/assets/m5_tee_nut.stl"/>
+      </geometry>
+    </collision>
+    <!-- Part m5_x_10mm_screw_5 -->
+    <visual>
+      <origin xyz="-0.464108 -1.48082 0.358683" rpy="1.55925 1.5708 0"/>
+      <geometry>
+        <mesh filename="package://robot_description/assets/m5_x_10mm_screw.stl"/>
+      </geometry>
+      <material name="m5_x_10mm_screw_5_material">
+        <color rgba="0.945098 0.94902 0.952941 1"/>
+      </material>
+    </visual>
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