Commit message: added degrees-of-freedome to the gantry

File: src/robot_description1/urdf/robot.urdf.xacro (robot description, xacro)
@@ -1971,10 +1971,10 @@
     </collision>
   </link>
-  <!-- Joint from leadscrew to z_axis_base -->
+  <!-- Joint from z_axis_base to leadscrew -->
   <joint name="z" type="prismatic">
-    <origin xyz="-0.119811 0.0001886 -0.823885" rpy="0 0 -0.0105398"/>
-    <parent link="leadscrew"/>
-    <child link="z_axis_base"/>
-    <axis xyz="0 0 1"/>
+    <origin xyz="0.119802 -0.00145135 0.823885" rpy="0 0 0.0105398"/>
+    <parent link="z_axis_base"/>
+    <child link="leadscrew"/>
+    <axis xyz="0 0 -1"/>
     <limit effort="10" velocity="10" lower="-1" upper="1"/>
   </joint>
@@ -2555,11 +2555,9 @@
     <limit effort="10" velocity="10" lower="-3.141592653589793" upper="3.141592653589793"/>
   </joint>
-  <!-- Joint from axis1 to leadscrew -->
-  <joint name="arm1" type="revolute">
-    <origin xyz="0.243812 -0.919886 1.65898" rpy="3.14159 0 1.5708"/>
-    <parent link="axis1"/>
-    <child link="leadscrew"/>
-    <axis xyz="0 0 1"/>
-    <limit effort="10" velocity="10" lower="-3.141592653589793" upper="3.141592653589793"/>
+  <!-- Joint from leadscrew to axis1 -->
+  <joint name="arm1" type="fixed">
+    <origin xyz="0.919921 -0.241288 1.65898" rpy="3.14159 0 1.5708"/>
+    <parent link="leadscrew"/>
+    <child link="axis1"/>
   </joint>
   <!-- Link axis2_4 -->
@@ -2723,11 +2721,11 @@
     <limit effort="10" velocity="10" lower="-3.141592653589793" upper="3.141592653589793"/>
   </joint>
-  <!-- Joint from body to axis1 -->
-  <joint name="extra_root_1_to_axis1" type="fixed">
-    <origin xyz="0 0 0" rpy="0 -0 0"/>
-    <parent link="body"/>
-    <child link="axis1"/>
-    <axis xyz="0 0 1"/>
-    <limit effort="10" velocity="10"/>
+  <!-- Joint from gantry_column to z_axis_base -->
+  <joint name="extra_root_1_to_axis1" type="prismatic">
+    <origin xyz="0.243999 -1.0397 2.48287" rpy="3.14159 0 1.58134"/>
+    <parent link="gantry_column"/>
+    <child link="z_axis_base"/>
+    <axis xyz="0 1 0"/>
+    <limit effort="10" velocity="10" lower="-1" upper="1"/>
   </joint>
   <!-- Link gantry_column -->
@@ -5684,10 +5682,10 @@
   </link>
   <!-- Joint from body to gantry_column -->
-  <joint name="extra_root_2_to_gantry_column" type="fixed">
+  <joint name="extra_root_2_to_gantry_column" type="prismatic">
     <origin xyz="0 0 0" rpy="0 -0 0"/>
     <parent link="body"/>
     <child link="gantry_column"/>
-    <axis xyz="0 0 1"/>
-    <limit effort="10" velocity="10"/>
+    <axis xyz="0 1 0"/>
+    <limit effort="10" velocity="10" lower="-1" upper="1"/>
   </joint>
 </robot>

Commit message: added collisions and fixed meshes paths

File: src/robot_description1/urdf/robot.urdf.xacro (robot description, xacro)
@@ -14,5 +14,5 @@
       <origin xyz="1.03456 -1.44349 0.368183" rpy="-0 -0 0.011542"/>
       <geometry>
-        <mesh filename="package://robot_description/assets/v_slot_20x40x1500_linear_rail.stl"/>
+        <mesh filename="package://robot_description1/meshes/v_slot_20x40x1500_linear_rail.stl"/>
       </geometry>
       <material name="v_slot_20x40x1500_linear_rail_material">
@@ -23,5 +23,5 @@
       <origin xyz="1.03456 -1.44349 0.368183" rpy="-0 -0 0.011542"/>
       <geometry>
-        <mesh filename="package://robot_description/assets/v_slot_20x40x1500_linear_rail.stl"/>
+        <mesh filename="package://robot_description1/meshes/v_slot_20x40x1500_linear_rail.stl"/>
       </geometry>
     </collision>
@@ -30,5 +30,5 @@
       <origin xyz="-0.45034 -1.46063 0.368183" rpy="-0 -0 0.011542"/>
       <geometry>
-        <mesh filename="package://robot_description/assets/v_slot_20x40x1500_linear_rail.stl"/>
+        <mesh filename="package://robot_description1/meshes/v_slot_20x40x1500_linear_rail.stl"/>
       </geometry>
       <material name="v_slot_20x40x1500_linear_rail_2_material">
@@ -39,5 +39,5 @@
       <origin xyz="-0.45034 -1.46063 0.368183" rpy="-0 -0 0.011542"/>
       <geometry>
-        <mesh filename="package://robot_description/assets/v_slot_20x40x1500_linear_rail.stl"/>
+        <mesh filename="package://robot_description1/meshes/v_slot_20x40x1500_linear_rail.stl"/>
       </geometry>
     </collision>
@@ -46,5 +46,5 @@
       <origin xyz="-0.467653 0.0392729 0.368183" rpy="-0 -0 0.011542"/>
       <geometry>
-        <mesh filename="package://robot_description/assets/v_slot_20x40x1500_linear_rail.stl"/>
+        <mesh filename="package://robot_description1/meshes/v_slot_20x40x1500_linear_rail.stl"/>
       </geometry>
       <material name="v_slot_20x40x1500_linear_rail_3_material">
@@ -55,5 +55,5 @@
       <origin xyz="-0.467653 0.0392729 0.368183" rpy="-0 -0 0.011542"/>
       <geometry>
-        <mesh filename="package://robot_description/assets/v_slot_20x40x1500_linear_rail.stl"/>
+        <mesh filename="package://robot_description1/meshes/v_slot_20x40x1500_linear_rail.stl"/>
       </geometry>
     </collision>
@@ -62,5 +62,5 @@
       <origin xyz="1.01725 0.0564124 0.368183" rpy="-0 -0 0.011542"/>
       <geometry>
-        <mesh filename="package://robot_description/assets/v_slot_20x40x1500_linear_rail.stl"/>
+        <mesh filename="package://robot_description1/meshes/v_slot_20x40x1500_linear_rail.stl"/>
       </geometry>
       <material name="v_slot_20x40x1500_linear_rail_4_material">
@@ -71,5 +71,5 @@
       <origin xyz="1.01725 0.0564124 0.368183" rpy="-0 -0 0.011542"/>
       <geometry>
-        <mesh filename="package://robot_description/assets/v_slot_20x40x1500_linear_rail.stl"/>
+        <mesh filename="package://robot_description1/meshes/v_slot_20x40x1500_linear_rail.stl"/>
       </geometry>
     </collision>
@@ -78,5 +78,5 @@
       <origin xyz="1.04857 -1.44393 0.358683" rpy="-1.5708 0 1.58234"/>
       <geometry>
-        <mesh filename="package://robot_description/assets/joining_plate_t.stl"/>
+        <mesh filename="package://robot_description1/meshes/joining_plate_t.stl"/>
       </geometry>
       <material name="joining_plate_t_material">
@@ -87,5 +87,5 @@
       <origin xyz="1.04857 -1.44393 0.358683" rpy="-1.5708 0 1.58234"/>
       <geometry>
-        <mesh filename="package://robot_description/assets/joining_plate_t.stl"/>
+        <mesh filename="package://robot_description1/meshes/joining_plate_t.stl"/>
       </geometry>
     </collision>
@@ -94,5 +94,5 @@
       <origin xyz="-0.464339 -1.46082 0.358683" rpy="-1.5708 -0 -1.55925"/>
       <geometry>
-        <mesh filename="package://robot_description/assets/joining_plate_t.stl"/>
+        <mesh filename="package://robot_description1/meshes/joining_plate_t.stl"/>
       </geometry>
       <material name="joining_plate_t_2_material">
@@ -103,5 +103,5 @@
       <origin xyz="-0.464339 -1.46082 0.358683" rpy="-1.5708 -0 -1.55925"/>
       <geometry>
-        <mesh filename="package://robot_description/assets/joining_plate_t.stl"/>
+        <mesh filename="package://robot_description1/meshes/joining_plate_t.stl"/>
       </geometry>
     </collision>
@@ -110,5 +110,5 @@
       <origin xyz="-0.477537 0.0291582 0.358683" rpy="-1.5708 0 1.58234"/>
       <geometry>
-        <mesh filename="package://robot_description/assets/joining_plate_90_degree.stl"/>
+        <mesh filename="package://robot_description1/meshes/joining_plate_90_degree.stl"/>
       </geometry>
       <material name="joining_plate_90_degree_material">
@@ -119,5 +119,5 @@
       <origin xyz="-0.477537 0.0291582 0.358683" rpy="-1.5708 0 1.58234"/>
       <geometry>
-        <mesh filename="package://robot_description/assets/joining_plate_90_degree.stl"/>
+        <mesh filename="package://robot_description1/meshes/joining_plate_90_degree.stl"/>
       </geometry>
     </collision>
@@ -126,5 +126,5 @@
       <origin xyz="-0.447142 -2.95069 0.358683" rpy="-1.5708 -0 -1.55925"/>
       <geometry>
-        <mesh filename="package://robot_description/assets/joining_plate_90_degree.stl"/>
+        <mesh filename="package://robot_description1/meshes/joining_plate_90_degree.stl"/>
       </geometry>
       <material name="joining_plate_90_degree_2_material">
@@ -135,5 +135,5 @@
       <origin xyz="-0.447142 -2.95069 0.358683" rpy="-1.5708 -0 -1.55925"/>
       <geometry>
-        <mesh filename="package://robot_description/assets/joining_plate_90_degree.stl"/>
+        <mesh filename="package://robot_description1/meshes/joining_plate_90_degree.stl"/>
       </geometry>
     </collision>
@@ -142,5 +142,5 @@
       <origin xyz="1.03776 -2.93355 0.358683" rpy="-1.5708 -0 -1.55925"/>
       <geometry>
-        <mesh filename="package://robot_description/assets/joining_plate_90_degree.stl"/>
+        <mesh filename="package://robot_description1/meshes/joining_plate_90_degree.stl"/>
       </geometry>
       <material name="joining_plate_90_degree_3_material">
@@ -151,5 +151,5 @@
       <origin xyz="1.03776 -2.93355 0.358683" rpy="-1.5708 -0 -1.55925"/>
       <geometry>
-        <mesh filename="package://robot_description/assets/joining_plate_90_degree.stl"/>
+        <mesh filename="package://robot_description1/meshes/joining_plate_90_degree.stl"/>
       </geometry>
     </collision>
@@ -158,5 +158,5 @@
       <origin xyz="1.03136 0.0465746 0.358683" rpy="-1.5708 0 1.58234"/>
       <geometry>
-        <mesh filename="package://robot_description/assets/joining_plate_90_degree.stl"/>
+        <mesh filename="package://robot_description1/meshes/joining_plate_90_degree.stl"/>
       </geometry>
       <material name="joining_plate_90_degree_4_material">
@@ -167,5 +167,5 @@
       <origin xyz="1.03136 0.0465746 0.358683" rpy="-1.5708 0 1.58234"/>
       <geometry>
-        <mesh filename="package://robot_description/assets/joining_plate_90_degree.stl"/>
+        <mesh filename="package://robot_description1/meshes/joining_plate_90_degree.stl"/>
       </geometry>
     </collision>
@@ -174,5 +174,5 @@
       <origin xyz="1.00736 0.0462976 0.358683" rpy="-1.5708 0 1.58234"/>
       <geometry>
-        <mesh filename="package://robot_description/assets/joining_plate_90_degree.stl"/>
+        <mesh filename="package://robot_description1/meshes/joining_plate_90_degree.stl"/>
       </geometry>
       <material name="joining_plate_90_degree_5_material">
@@ -183,5 +183,5 @@
       <origin xyz="1.00736 0.0462976 0.358683" rpy="-1.5708 0 1.58234"/>
       <geometry>
-        <mesh filename="package://robot_description/assets/joining_plate_90_degree.stl"/>
+        <mesh filename="package://robot_description1/meshes/joining_plate_90_degree.stl"/>
       </geometry>
     </collision>
@@ -190,5 +190,5 @@
       <origin xyz="-0.423144 -2.95041 0.358683" rpy="-1.5708 -0 -1.55925"/>
       <geometry>
-        <mesh filename="package://robot_description/assets/joining_plate_90_degree.stl"/>
+        <mesh filename="package://robot_description1/meshes/joining_plate_90_degree.stl"/>
       </geometry>
       <material name="joining_plate_90_degree_6_material">
@@ -199,5 +199,5 @@
       <origin xyz="-0.423144 -2.95041 0.358683" rpy="-1.5708 -0 -1.55925"/>
       <geometry>
-        <mesh filename="package://robot_description/assets/joining_plate_90_degree.stl"/>
+        <mesh filename="package://robot_description1/meshes/joining_plate_90_degree.stl"/>
       </geometry>
     </collision>
@@ -206,5 +206,5 @@
       <origin xyz="-0.453539 0.0294352 0.358683" rpy="-1.5708 0 1.58234"/>
       <geometry>
-        <mesh filename="package://robot_description/assets/joining_plate_90_degree.stl"/>
+        <mesh filename="package://robot_description1/meshes/joining_plate_90_degree.stl"/>
       </geometry>
       <material name="joining_plate_90_degree_7_material">
@@ -215,5 +215,5 @@
       <origin xyz="-0.453539 0.0294352 0.358683" rpy="-1.5708 0 1.58234"/>
       <geometry>
-        <mesh filename="package://robot_description/assets/joining_plate_90_degree.stl"/>
+        <mesh filename="package://robot_description1/meshes/joining_plate_90_degree.stl"/>
       </geometry>
     </collision>
@@ -222,5 +222,5 @@
       <origin xyz="1.06176 -2.93327 0.358683" rpy="-1.5708 -0 -1.55925"/>
       <geometry>
-        <mesh filename="package://robot_description/assets/joining_plate_90_degree.stl"/>
+        <mesh filename="package://robot_description1/meshes/joining_plate_90_degree.stl"/>
       </geometry>
       <material name="joining_plate_90_degree_8_material">
@@ -231,5 +231,5 @@
       <origin xyz="1.06176 -2.93327 0.358683" rpy="-1.5708 -0 -1.55925"/>
       <geometry>
-        <mesh filename="package://robot_description/assets/joining_plate_90_degree.stl"/>
+        <mesh filename="package://robot_description1/meshes/joining_plate_90_degree.stl"/>
       </geometry>
     </collision>
@@ -238,5 +238,5 @@
       <origin xyz="1.03927 -1.44403 0.358683" rpy="-1.58234 1.5708 0"/>
       <geometry>
-        <mesh filename="package://robot_description/assets/m5_tee_nut.stl"/>
+        <mesh filename="package://robot_description1/meshes/m5_tee_nut.stl"/>
       </geometry>
       <material name="m5_tee_nut_material">
@@ -247,5 +247,5 @@
       <origin xyz="1.03927 -1.44403 0.358683" rpy="-1.58234 1.5708 0"/>
       <geometry>
-        <mesh filename="package://robot_description/assets/m5_tee_nut.stl"/>
+        <mesh filename="package://robot_description1/meshes/m5_tee_nut.stl"/>
       </geometry>
     </collision>
@@ -254,5 +254,5 @@
       <origin xyz="1.04857 -1.44393 0.358683" rpy="-1.58234 1.5708 0"/>
       <geometry>
-        <mesh filename="package://robot_description/assets/m5_x_10mm_screw.stl"/>
+        <mesh filename="package://robot_description1/meshes/m5_x_10mm_screw.stl"/>
       </geometry>
       <material name="m5_x_10mm_screw_material">
@@ -263,5 +263,5 @@
       <origin xyz="1.04857 -1.44393 0.358683" rpy="-1.58234 1.5708 0"/>
       <geometry>
-        <mesh filename="package://robot_description/assets/m5_x_10mm_screw.stl"/>
+        <mesh filename="package://robot_description1/meshes/m5_x_10mm_screw.stl"/>
       </geometry>
     </collision>
@@ -270,5 +270,5 @@
       <origin xyz="1.03904 -1.42403 0.358683" rpy="-1.58234 1.5708 0"/>
       <geometry>
-        <mesh filename="package://robot_description/assets/m5_tee_nut.stl"/>
+        <mesh filename="package://robot_description1/meshes/m5_tee_nut.stl"/>
       </geometry>
       <material name="m5_tee_nut_2_material">
@@ -279,5 +279,5 @@
       <origin xyz="1.03904 -1.42403 0.358683" rpy="-1.58234 1.5708 0"/>
       <geometry>
-        <mesh filename="package://robot_description/assets/m5_tee_nut.stl"/>
+        <mesh filename="package://robot_description1/meshes/m5_tee_nut.stl"/>
       </geometry>
     </collision>
@@ -286,5 +286,5 @@
       <origin xyz="1.04834 -1.42393 0.358683" rpy="-1.58234 1.5708 0"/>
       <geometry>
-        <mesh filename="package://robot_description/assets/m5_x_10mm_screw.stl"/>
+        <mesh filename="package://robot_description1/meshes/m5_x_10mm_screw.stl"/>
       </geometry>
       <material name="m5_x_10mm_screw_2_material">
@@ -295,5 +295,5 @@
       <origin xyz="1.04834 -1.42393 0.358683" rpy="-1.58234 1.5708 0"/>
       <geometry>
-        <mesh filename="package://robot_description/assets/m5_x_10mm_screw.stl"/>
+        <mesh filename="package://robot_description1/meshes/m5_x_10mm_screw.stl"/>
       </geometry>
     </collision>
@@ -302,5 +302,5 @@
       <origin xyz="1.0395 -1.46403 0.358683" rpy="-1.58234 1.5708 0"/>
       <geometry>
-        <mesh filename="package://robot_description/assets/m5_tee_nut.stl"/>
+        <mesh filename="package://robot_description1/meshes/m5_tee_nut.stl"/>
       </geometry>
       <material name="m5_tee_nut_3_material">
@@ -311,5 +311,5 @@
       <origin xyz="1.0395 -1.46403 0.358683" rpy="-1.58234 1.5708 0"/>
       <geometry>
-        <mesh filename="package://robot_description/assets/m5_tee_nut.stl"/>
+        <mesh filename="package://robot_description1/meshes/m5_tee_nut.stl"/>
       </geometry>
     </collision>
@@ -318,5 +318,5 @@
       <origin xyz="1.0488 -1.46392 0.358683" rpy="-1.58234 1.5708 0"/>
       <geometry>
-        <mesh filename="package://robot_description/assets/m5_x_10mm_screw.stl"/>
+        <mesh filename="package://robot_description1/meshes/m5_x_10mm_screw.stl"/>
       </geometry>
       <material name="m5_x_10mm_screw_3_material">
@@ -327,5 +327,5 @@
       <origin xyz="1.0488 -1.46392 0.358683" rpy="-1.58234 1.5708 0"/>
       <geometry>
-        <mesh filename="package://robot_description/assets/m5_x_10mm_screw.stl"/>
+        <mesh filename="package://robot_description1/meshes/m5_x_10mm_screw.stl"/>
       </geometry>
     </collision>
@@ -334,5 +334,5 @@
       <origin xyz="-0.45504 -1.46071 0.358683" rpy="1.55925 1.5708 0"/>
       <geometry>
-        <mesh filename="package://robot_description/assets/m5_tee_nut.stl"/>
+        <mesh filename="package://robot_description1/meshes/m5_tee_nut.stl"/>
       </geometry>
       <material name="m5_tee_nut_4_material">
@@ -343,5 +343,5 @@
       <origin xyz="-0.45504 -1.46071 0.358683" rpy="1.55925 1.5708 0"/>
       <geometry>
-        <mesh filename="package://robot_description/assets/m5_tee_nut.stl"/>
+        <mesh filename="package://robot_description1/meshes/m5_tee_nut.stl"/>
       </geometry>
     </collision>
@@ -350,5 +350,5 @@
       <origin xyz="-0.464339 -1.46082 0.358683" rpy="1.55925 1.5708 0"/>
       <geometry>
-        <mesh filename="package://robot_description/assets/m5_x_10mm_screw.stl"/>
+        <mesh filename="package://robot_description1/meshes/m5_x_10mm_screw.stl"/>
       </geometry>
       <material name="m5_x_10mm_screw_4_material">
@@ -359,5 +359,5 @@
       <origin xyz="-0.464339 -1.46082 0.358683" rpy="1.55925 1.5708 0"/>
       <geometry>
-        <mesh filename="package://robot_description/assets/m5_x_10mm_screw.stl"/>
+        <mesh filename="package://robot_description1/meshes/m5_x_10mm_screw.stl"/>
       </geometry>
     </collision>
@@ -366,5 +366,5 @@
       <origin xyz="-0.454809 -1.48071 0.358683" rpy="1.55925 1.5708 0"/>
       <geometry>
-        <mesh filename="package://robot_description/assets/m5_tee_nut.stl"/>
+        <mesh filename="package://robot_description1/meshes/m5_tee_nut.stl"/>
       </geometry>
       <material name="m5_tee_nut_5_material">
@@ -375,5 +375,5 @@
       <origin xyz="-0.454809 -1.48071 0.358683" rpy="1.55925 1.5708 0"/>
       <geometry>
-        <mesh filename="package://robot_description/assets/m5_tee_nut.stl"/>
+        <mesh filename="package://robot_description1/meshes/m5_tee_nut.stl"/>
       </geometry>
     </collision>
@@ -382,5 +382,5 @@
       <origin xyz="-0.464108 -1.48082 0.358683" rpy="1.55925 1.5708 0"/>
       <geometry>
-        <mesh filename="package://robot_description/assets/m5_x_10mm_screw.stl"/>
+        <mesh filename="package://robot_description1/meshes/m5_x_10mm_screw.stl"/>
       </geometry>
       <material name="m5_x_10mm_screw_5_material">
@@ -391,5 +391,5 @@
       <origin xyz="-0.464108 -1.48082 0.358683" rpy="1.55925 1.5708 0"/>
       <geometry>
-        <mesh filename="package://robot_description/assets/m5_x_10mm_screw.stl"/>
+        <mesh filename="package://robot_description1/meshes/m5_x_10mm_screw.stl"/>
       </geometry>
     </collision>
@@ -398,5 +398,5 @@
       <origin xyz="-0.455271 -1.44072 0.358683" rpy="1.55925 1.5708 0"/>
       <geometry>
-        <mesh filename="package://robot_description/assets/m5_tee_nut.stl"/>
+        <mesh filename="package://robot_description1/meshes/m5_tee_nut.stl"/>
       </geometry>
       <material name="m5_tee_nut_6_material">
@@ -407,5 +407,5 @@
       <origin xyz="-0.455271 -1.44072 0.358683" rpy="1.55925 1.5708 0"/>
       <geometry>
-        <mesh filename="package://robot_description/assets/m5_tee_nut.stl"/>
+        <mesh filename="package://robot_description1/meshes/m5_tee_nut.stl"/>
       </geometry>
     </collision>
@@ -414,5 +414,5 @@
       <origin xyz="-0.46457 -1.44082 0.358683" rpy="1.55925 1.5708 0"/>
       <geometry>
-        <mesh filename="package://robot_description/assets/m5_x_10mm_screw.stl"/>
+        <mesh filename="package://robot_description1/meshes/m5_x_10mm_screw.stl"/>
       </geometry>
       <material name="m5_x_10mm_screw_6_material">
@@ -423,5 +423,5 @@
       <origin xyz="-0.46457 -1.44082 0.358683" rpy="1.55925 1.5708 0"/>
       <geometry>
-        <mesh filename="package://robot_description/assets/m5_x_10mm_screw.stl"/>
+        <mesh filename="package://robot_description1/meshes/m5_x_10mm_screw.stl"/>
       </geometry>
     </collision>
@@ -430,5 +430,5 @@
       <origin xyz="-0.472006 0.00922067 0.358683" rpy="3.14159 0 1.58234"/>
       <geometry>
-        <mesh filename="package://robot_description/assets/m5_tee_nut.stl"/>
+        <mesh filename="package://robot_description1/meshes/m5_tee_nut.stl"/>
       </geometry>
       <material name="m5_tee_nut_7_material">
@@ -439,5 +439,5 @@
       <origin xyz="-0.472006 0.00922067 0.358683" rpy="3.14159 0 1.58234"/>
       <geometry>
-        <mesh filename="package://robot_description/assets/m5_tee_nut.stl"/>
+        <mesh filename="package://robot_description1/meshes/m5_tee_nut.stl"/>
       </geometry>
     </collision>
@@ -446,5 +446,5 @@
       <origin xyz="-0.481306 0.00911333 0.358683" rpy="3.14159 0 1.58234"/>
       <geometry>
-        <mesh filename="package://robot_description/assets/m5_x_10mm_screw.stl"/>
+        <mesh filename="package://robot_description1/meshes/m5_x_10mm_screw.stl"/>
       </geometry>
       <material name="m5_x_10mm_screw_7_material">
@@ -455,5 +455,5 @@
       <origin xyz="-0.481306 0.00911333 0.358683" rpy="3.14159 0 1.58234"/>
       <geometry>
-        <mesh filename="package://robot_description/assets/m5_x_10mm_screw.stl"/>
+        <mesh filename="package://robot_description1/meshes/m5_x_10mm_screw.stl"/>
       </geometry>
     </collision>
@@ -462,5 +462,5 @@
       <origin xyz="-0.471776 -0.010778 0.358683" rpy="3.14159 0 1.58234"/>
       <geometry>
-        <mesh filename="package://robot_description/assets/m5_tee_nut.stl"/>
+        <mesh filename="package://robot_description1/meshes/m5_tee_nut.stl"/>
       </geometry>
       <material name="m5_tee_nut_8_material">
@@ -471,5 +471,5 @@
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