Commit message: added collisions and fixed meshes paths

File: src/robot_description2/urdf/dual_roarm.urdf.xacro (robot description, xacro)
@@ -16,4 +16,9 @@
       <material name="gray"/>
     </visual>
+    <collision>
+      <geometry>
+        <box size="1.0 0.5 0.02"/>
+      </geometry>
+    </collision>
   </link>
   <joint name="world_to_mounting_plate" type="fixed">
@@ -31,4 +36,10 @@
         <material name="gray"/>
       </visual>
+      <collision>
+        <geometry>
+          <mesh filename="package://roarm/meshes/base.stl"/>
+        </geometry>
+        <origin rpy="0 0 0" xyz="0 0 0"/>
+      </collision>
     </link>
     <joint name="${prefix}world_to_base" type="fixed">
@@ -45,4 +56,10 @@
         <material name="white"/>
       </visual>
+      <collision>
+        <geometry>
+          <mesh filename="package://roarm/meshes/L1.stl"/>
+        </geometry>
+        <origin rpy="0 0 0" xyz="0 0 -0.062"/>
+      </collision>
     </link>
     <link name="${prefix}l2_link">
@@ -54,4 +71,10 @@
         <material name="white"/>
       </visual>
+      <collision>
+        <geometry>
+          <mesh filename="package://roarm/meshes/L2.stl"/>
+        </geometry>
+        <origin rpy="0 0 0" xyz="0 -0.041051 -0.11574"/>
+      </collision>
     </link>
     <link name="${prefix}l3_link">
@@ -63,4 +86,10 @@
         <material name="white"/>
       </visual>
+      <collision>
+        <geometry>
+          <mesh filename="package://roarm/meshes/L3.stl"/>
+        </geometry>
+        <origin rpy="0 0 0" xyz="0 -0.160452 -0.235141"/>
+      </collision>
     </link>
     <link name="${prefix}l4_link">
@@ -72,4 +101,10 @@
         <material name="white"/>
       </visual>
+      <collision>
+        <geometry>
+          <mesh filename="package://roarm/meshes/L4.stl"/>
+        </geometry>
+        <origin rpy="0 0 0" xyz="0 -0.250907 -0.325596"/>
+      </collision>
     </link>
     <link name="${prefix}l5_1_A_link">
@@ -81,4 +116,10 @@
         <material name="white"/>
       </visual>
+      <collision>
+        <geometry>
+          <mesh filename="package://roarm/meshes/L5_1_A.stl"/>
+        </geometry>
+        <origin xyz="-0.003489 -0.311007 -0.358744" rpy="0 0 0"/>
+      </collision>
     </link>
     <link name="${prefix}l5_1_B_link">
@@ -90,4 +131,10 @@
         <material name="white"/>
       </visual>
+      <collision>
+        <geometry>
+          <mesh filename="package://roarm/meshes/L5_1_B.stl"/>
+        </geometry>
+        <origin xyz="-0.024489 -0.311007 -0.358744" rpy="0 0 0"/>
+      </collision>
     </link>
     <link name="${prefix}l5_2_A_link">
@@ -99,4 +146,10 @@
         <material name="white"/>
       </visual>
+      <collision>
+        <geometry>
+          <mesh filename="package://roarm/meshes/L5_2_A.stl"/>
+        </geometry>
+        <origin xyz="0.017511 -0.285551 -0.362001" rpy="0 0 0"/>
+      </collision>
     </link>
     <link name="${prefix}l5_2_B_link">
@@ -108,4 +161,10 @@
         <material name="white"/>
       </visual>
+      <collision>
+        <geometry>
+          <mesh filename="package://roarm/meshes/L5_2_B.stl"/>
+        </geometry>
+        <origin xyz="-0.045489 -0.285551 -0.362001" rpy="0 0 0"/>
+      </collision>
     </link>
     <link name="${prefix}l5_3_A_link">
@@ -117,4 +176,10 @@
         <material name="white"/>
       </visual>
+      <collision>
+        <geometry>
+          <mesh filename="package://roarm/meshes/L5_3_A.stl"/>
+        </geometry>
+        <origin xyz="0.039711 -0.304219 -0.347532" rpy="0 0 0"/>
+      </collision>
     </link>
     <link name="${prefix}l5_3_B_link">
@@ -126,4 +191,10 @@
         <material name="white"/>
       </visual>
+      <collision>
+        <geometry>
+          <mesh filename="package://roarm/meshes/L5_3_B.stl"/>
+        </geometry>
+        <origin xyz="-0.067689 -0.304219 -0.347532" rpy="0 0 0"/>
+      </collision>
     </link>
     <joint name="${prefix}base_to_L1" type="revolute">

Commit message: fixed urdf

File: src/robot_description1/urdf/robot.urdf.xacro (robot description, xacro)
@@ -3,4 +3,6 @@
 <!-- Onshape https://cad.onshape.com/documents/a2e4d90d4720e7eb81b47647/w/f29fb00f1617a93c8228a45a/e/5adbd4e56813ca0b03de2f98 -->
 <robot name="onshape-to-robot">
+  <!-- Explicit world frame so RViz Fixed Frame 'world' resolves -->
+  <link name="world"/>
   <!-- Link body -->
   <link name="body">
@@ -1195,4 +1197,10 @@
     </collision>
   </link>
+  <!-- Anchor the robot model to world -->
+  <joint name="world_to_body" type="fixed">
+    <origin xyz="0 0 0" rpy="0 0 0"/>
+    <parent link="world"/>
+    <child link="body"/>
+  </joint>
   <!-- Link axis1 -->
   <link name="axis1">

Commit message: rename joints

File: src/robot_description1/urdf/robot.urdf.xacro (robot description, xacro)
@@ -2132,5 +2132,5 @@
   </link>
   <!-- Joint from axis5 to axis6 -->
-  <joint name="joint5 (1)" type="revolute">
+  <joint name="arm2_joint5" type="revolute">
     <origin xyz="-0 0.11 -0.03" rpy="-1.5708 -1.54613 -3.14159"/>
     <parent link="axis5"/>
@@ -2140,5 +2140,5 @@
   </joint>
   <!-- Joint from axis4 to axis5 -->
-  <joint name="joint4 (1)" type="revolute">
+  <joint name="arm2_joint4" type="revolute">
     <origin xyz="0 -0.005 -0.09" rpy="-1.5708 -1.46178 -3.14159"/>
     <parent link="axis4"/>
@@ -2148,5 +2148,5 @@
   </joint>
   <!-- Joint from axis3 to axis4 -->
-  <joint name="joint3 (1)" type="revolute">
+  <joint name="arm2_joint3" type="revolute">
     <origin xyz="0.000135636 -0.19 0.03" rpy="-1.5708 0.529841 -0"/>
     <parent link="axis3"/>
@@ -2156,5 +2156,5 @@
   </joint>
   <!-- Joint from axis2 to axis3 -->
-  <joint name="joint2 (1)" type="revolute">
+  <joint name="arm2_joint2" type="revolute">
     <origin xyz="0 0.15 -0.02" rpy="-3.14159 0 1.2109"/>
     <parent link="axis2"/>
@@ -2164,5 +2164,5 @@
   </joint>
   <!-- Joint from axis1_2 to axis2 -->
-  <joint name="joint1 (1)" type="revolute">
+  <joint name="arm2_joint1" type="revolute">
     <origin xyz="0 0 -0.18" rpy="1.5708 -1.17344 1.5708"/>
     <parent link="axis1_2"/>
@@ -2172,5 +2172,5 @@
   </joint>
   <!-- Joint from leadscrew to axis1_2 -->
-  <joint name="arm2" type="revolute">
+  <joint name="arm2_joint0" type="revolute">
     <origin xyz="-0.12 0.17 0" rpy="-3.14159 0 0"/>
     <parent link="leadscrew"/>
@@ -2324,5 +2324,5 @@
   </link>
   <!-- Joint from axis5_2 to axis6_2 -->
-  <joint name="joint5 (1) (1)" type="revolute">
+  <joint name="arm3_joint5" type="revolute">
     <origin xyz="-0 0.11 -0.03" rpy="-1.5708 -0.938431 3.14159"/>
     <parent link="axis5_2"/>
@@ -2332,5 +2332,5 @@
   </joint>
   <!-- Joint from axis4_2 to axis5_2 -->
-  <joint name="joint4 (1) (1)" type="revolute">
+  <joint name="arm3_joint4" type="revolute">
     <origin xyz="0 -0.005 -0.09" rpy="-1.5708 -0.555692 3.14159"/>
     <parent link="axis4_2"/>
@@ -2340,5 +2340,5 @@
   </joint>
   <!-- Joint from axis3_2 to axis4_2 -->
-  <joint name="joint3 (1) (1)" type="revolute">
+  <joint name="arm3_joint3" type="revolute">
     <origin xyz="0.000135636 -0.19 0.03" rpy="1.5708 1.52901 -3.14159"/>
     <parent link="axis3_2"/>
@@ -2348,5 +2348,5 @@
   </joint>
   <!-- Joint from axis2_2 to axis3_2 -->
-  <joint name="joint2 (1) (1)" type="revolute">
+  <joint name="arm3_joint2" type="revolute">
     <origin xyz="-0 0.15 -0.02" rpy="-3.14159 0 1.42829"/>
     <parent link="axis2_2"/>
@@ -2356,5 +2356,5 @@
   </joint>
   <!-- Joint from axis1_3 to axis2_2 -->
-  <joint name="joint1 (1) (1)" type="revolute">
+  <joint name="arm3_joint1" type="revolute">
     <origin xyz="-0 0 -0.18" rpy="1.5708 -1.17344 -0.163809"/>
     <parent link="axis1_3"/>
@@ -2364,5 +2364,5 @@
   </joint>
   <!-- Joint from leadscrew to axis1_3 -->
-  <joint name="arm3" type="revolute">
+  <joint name="arm3_joint0" type="revolute">
     <origin xyz="-0.24 -0 0" rpy="-3.14159 0 0"/>
     <parent link="leadscrew"/>
@@ -2516,5 +2516,5 @@
   </link>
   <!-- Joint from axis5_3 to axis6_3 -->
-  <joint name="joint5 (2)" type="revolute">
+  <joint name="arm4_joint5" type="revolute">
     <origin xyz="-0 0.11 -0.03" rpy="1.5708 -0.581164 -0"/>
     <parent link="axis5_3"/>
@@ -2524,5 +2524,5 @@
   </joint>
   <!-- Joint from axis4_3 to axis5_3 -->
-  <joint name="joint4 (2)" type="revolute">
+  <joint name="arm4_joint4" type="revolute">
     <origin xyz="0 -0.005 -0.09" rpy="-1.5708 -1.40423 3.14159"/>
     <parent link="axis4_3"/>
@@ -2532,5 +2532,5 @@
   </joint>
   <!-- Joint from axis3_3 to axis4_3 -->
-  <joint name="joint3 (2)" type="revolute">
+  <joint name="arm4_joint3" type="revolute">
     <origin xyz="0.000135636 -0.19 0.03" rpy="-1.5708 -0.640792 -0"/>
     <parent link="axis3_3"/>
@@ -2540,5 +2540,5 @@
   </joint>
   <!-- Joint from axis2_3 to axis3_3 -->
-  <joint name="joint2 (2)" type="revolute">
+  <joint name="arm4_joint2" type="revolute">
     <origin xyz="0 0.15 -0.02" rpy="3.14159 0 1.2109"/>
     <parent link="axis2_3"/>
@@ -2548,5 +2548,5 @@
   </joint>
   <!-- Joint from axis1_4 to axis2_3 -->
-  <joint name="joint1 (2)" type="revolute">
+  <joint name="arm4_joint1" type="revolute">
     <origin xyz="0 0 -0.18" rpy="1.5708 -1.17344 -1.5708"/>
     <parent link="axis1_4"/>
@@ -2556,5 +2556,5 @@
   </joint>
   <!-- Joint from leadscrew to axis1_4 -->
-  <joint name="arm4" type="revolute">
+  <joint name="arm4_joint0" type="revolute">
     <origin xyz="-0.12 -0.17 0" rpy="-3.14159 0 0"/>
     <parent link="leadscrew"/>
@@ -2564,5 +2564,5 @@
   </joint>
   <!-- Joint from leadscrew to axis1 -->
-  <joint name="arm1" type="fixed">
+  <joint name="arm1_joint0" type="fixed">
     <origin xyz="0.919921 -0.241288 1.65898" rpy="3.14159 0 1.5708"/>
     <parent link="leadscrew"/>
@@ -2690,5 +2690,5 @@
   </link>
   <!-- Joint from axis5_4 to axis6_4 -->
-  <joint name="joint5" type="revolute">
+  <joint name="arm1_joint5" type="revolute">
     <origin xyz="0 0.11 -0.03" rpy="-1.5708 -1.54613 -3.14159"/>
     <parent link="axis5_4"/>
@@ -2698,5 +2698,5 @@
   </joint>
   <!-- Joint from axis4_4 to axis5_4 -->
-  <joint name="joint4" type="revolute">
+  <joint name="arm1_joint4" type="revolute">
     <origin xyz="0 -0.005 -0.09" rpy="-1.5708 -1.46178 3.14159"/>
     <parent link="axis4_4"/>
@@ -2706,5 +2706,5 @@
   </joint>
   <!-- Joint from axis3_4 to axis4_4 -->
-  <joint name="joint3" type="revolute">
+  <joint name="arm1_joint3" type="revolute">
     <origin xyz="0.000135636 -0.19 0.03" rpy="-1.5708 0.529841 -0"/>
     <parent link="axis3_4"/>
@@ -2714,5 +2714,5 @@
   </joint>
   <!-- Joint from axis2_4 to axis3_4 -->
-  <joint name="joint2" type="revolute">
+  <joint name="arm1_joint2" type="revolute">
     <origin xyz="0 0.15 -0.02" rpy="-3.14159 -0 1.2109"/>
     <parent link="axis2_4"/>
@@ -2722,5 +2722,5 @@
   </joint>
   <!-- Joint from axis1 to axis2_4 -->
-  <joint name="joint1" type="revolute">
+  <joint name="arm1_joint1" type="revolute">
     <origin xyz="0.243812 -0.919886 1.47898" rpy="1.5708 -1.17344 -1.5708"/>
     <parent link="axis1"/>

Commit message: wip: trying to load gazebo simulation

File: src/robot_description1/urdf/robot.urdf.xacro (robot description, xacro)
@@ -1619,4 +1619,49 @@
     </collision>
   </link>
+  <!-- Camera mounted below the z_axis_bottom assembly -->
+  <link name="z_bottom_camera_link">
+    <inertial>
+      <origin xyz="0 0 0" rpy="0 0 0"/>
+      <mass value="1e-06"/>
+      <inertia ixx="1e-06" ixy="0" ixz="0" iyy="1e-06" iyz="0" izz="1e-06"/>
+    </inertial>
+  </link>
+  <link name="z_bottom_camera_optical_frame">
+    <inertial>
+      <origin xyz="0 0 0" rpy="0 0 0"/>
+      <mass value="1e-06"/>
+      <inertia ixx="1e-06" ixy="0" ixz="0" iyy="1e-06" iyz="0" izz="1e-06"/>
+    </inertial>
+  </link>
+  <joint name="z_bottom_camera_joint" type="fixed">
+    <origin xyz="-0.12 0 -0.06" rpy="0 0 0"/>
+    <parent link="leadscrew"/>
+    <child link="z_bottom_camera_link"/>
+  </joint>
+  <joint name="z_bottom_camera_optical_joint" type="fixed">
+    <origin xyz="0 0 0" rpy="-1.57079632679 0 -1.57079632679"/>
+    <parent link="z_bottom_camera_link"/>
+    <child link="z_bottom_camera_optical_frame"/>
+  </joint>
+  <gazebo reference="z_bottom_camera_link">
+    <sensor name="z_bottom_camera" type="camera">
+      <always_on>true</always_on>
+      <update_rate>30</update_rate>
+      <visualize>true</visualize>
+      <topic>/z_bottom_camera/image_raw</topic>
+      <camera name="z_bottom_camera_sensor">
+        <horizontal_fov>1.047</horizontal_fov>
+        <image>
+          <width>1280</width>
+          <height>720</height>
+          <format>R8G8B8</format>
+        </image>
+        <clip>
+          <near>0.02</near>
+          <far>10.0</far>
+        </clip>
+      </camera>
+    </sensor>
+  </gazebo>
   <!-- Link z_axis_base -->
   <link name="z_axis_base">
