Commit message: masses and inertias and simpler collision primitives

File: src/robot_description1/urdf/robot.urdf.xacro (robot description, xacro)
@@ -9,6 +9,6 @@
     <inertial>
       <origin xyz="0 0 0" rpy="0 0 0"/>
-      <mass value="1e-09"/>
-      <inertia ixx="1e-09" ixy="0" ixz="0" iyy="1e-09" iyz="0" izz="1e-09"/>
+      <mass value="45.0"/>
+      <inertia ixx="33.80" ixy="0" ixz="0" iyy="9.65" iyz="0" izz="43.35"/>
     </inertial>
     <!-- Part v_slot_20x40x1500_linear_rail -->
@@ -1207,6 +1207,6 @@
     <inertial>
       <origin xyz="0 0 0" rpy="0 0 0"/>
-      <mass value="1e-09"/>
-      <inertia ixx="1e-09" ixy="0" ixz="0" iyy="1e-09" iyz="0" izz="1e-09"/>
+      <mass value="0.25"/>
+      <inertia ixx="8.33e-05" ixy="0" ixz="0" iyy="8.33e-05" iyz="0" izz="1.50e-04"/>
     </inertial>
     <!-- Part axis1 -->
@@ -1223,5 +1223,5 @@
       <origin xyz="0.238812 -0.949886 1.64898" rpy="-0 0 1.5708"/>
       <geometry>
-        <mesh filename="package://robot_description1/meshes/axis1.stl"/>
+        <box size="0.06 0.06 0.02"/>
       </geometry>
     </collision>
@@ -1231,6 +1231,6 @@
     <inertial>
       <origin xyz="0 0 0" rpy="0 0 0"/>
-      <mass value="1e-09"/>
-      <inertia ixx="1e-09" ixy="0" ixz="0" iyy="1e-09" iyz="0" izz="1e-09"/>
+      <mass value="8.0"/>
+      <inertia ixx="0.628" ixy="0" ixz="0" iyy="0.643" iyz="0" izz="0.068"/>
     </inertial>
     <!-- Part precision_rod_d10mm_l800mm -->
@@ -1668,6 +1668,6 @@
     <inertial>
       <origin xyz="0 0 0" rpy="0 0 0"/>
-      <mass value="1e-09"/>
-      <inertia ixx="1e-09" ixy="0" ixz="0" iyy="1e-09" iyz="0" izz="1e-09"/>
+      <mass value="3.0"/>
+      <inertia ixx="0.0117" ixy="0" ixz="0" iyy="0.0157" iyz="0" izz="0.0202"/>
     </inertial>
     <!-- Part linear_bearing_lm10uu -->
@@ -2036,6 +2036,6 @@
     <inertial>
       <origin xyz="0 0 0" rpy="0 0 0"/>
-      <mass value="1e-09"/>
-      <inertia ixx="1e-09" ixy="0" ixz="0" iyy="1e-09" iyz="0" izz="1e-09"/>
+      <mass value="0.25"/>
+      <inertia ixx="8.33e-05" ixy="0" ixz="0" iyy="8.33e-05" iyz="0" izz="1.50e-04"/>
     </inertial>
     <!-- Part axis1_2 -->
@@ -2052,5 +2052,5 @@
       <origin xyz="0.005 0.03 -0.01" rpy="-0 -0 -1.5708"/>
       <geometry>
-        <mesh filename="package://robot_description1/meshes/axis1.stl"/>
+        <box size="0.06 0.06 0.02"/>
       </geometry>
     </collision>
@@ -2060,6 +2060,6 @@
     <inertial>
       <origin xyz="0 0 0" rpy="0 0 0"/>
-      <mass value="1e-09"/>
-      <inertia ixx="1e-09" ixy="0" ixz="0" iyy="1e-09" iyz="0" izz="1e-09"/>
+      <mass value="0.20"/>
+      <inertia ixx="5.67e-05" ixy="0" ixz="0" iyy="5.67e-05" iyz="0" izz="8.33e-05"/>
     </inertial>
     <!-- Part axis2 -->
@@ -2076,5 +2076,5 @@
       <origin xyz="-0.025 -0.025 -0.015" rpy="1.5708 -0 0"/>
       <geometry>
-        <mesh filename="package://robot_description1/meshes/axis2.stl"/>
+        <box size="0.05 0.05 0.03"/>
       </geometry>
     </collision>
@@ -2084,6 +2084,6 @@
     <inertial>
       <origin xyz="0 0 0" rpy="0 0 0"/>
-      <mass value="1e-09"/>
-      <inertia ixx="1e-09" ixy="0" ixz="0" iyy="1e-09" iyz="0" izz="1e-09"/>
+      <mass value="0.18"/>
+      <inertia ixx="4.80e-05" ixy="0" ixz="0" iyy="6.15e-05" iyz="0" izz="6.15e-05"/>
     </inertial>
     <!-- Part axis3 -->
@@ -2100,5 +2100,5 @@
       <origin xyz="-0.0201356 0.02 0.025" rpy="-1.5708 -0 -0"/>
       <geometry>
-        <mesh filename="package://robot_description1/meshes/axis3.stl"/>
+        <box size="0.05 0.04 0.04"/>
       </geometry>
     </collision>
@@ -2108,6 +2108,6 @@
     <inertial>
       <origin xyz="0 0 0" rpy="0 0 0"/>
-      <mass value="1e-09"/>
-      <inertia ixx="1e-09" ixy="0" ixz="0" iyy="1e-09" iyz="0" izz="1e-09"/>
+      <mass value="0.15"/>
+      <inertia ixx="3.13e-05" ixy="0" ixz="0" iyy="4.25e-05" iyz="0" izz="5.13e-05"/>
     </inertial>
     <!-- Part axis4 -->
@@ -2124,5 +2124,5 @@
       <origin xyz="-0.02 0.005 -0.02" rpy="0 -0 0"/>
       <geometry>
-        <mesh filename="package://robot_description1/meshes/axis4.stl"/>
+        <box size="0.05 0.04 0.03"/>
       </geometry>
     </collision>
@@ -2132,6 +2132,6 @@
     <inertial>
       <origin xyz="0 0 0" rpy="0 0 0"/>
-      <mass value="1e-09"/>
-      <inertia ixx="1e-09" ixy="0" ixz="0" iyy="1e-09" iyz="0" izz="1e-09"/>
+      <mass value="0.14"/>
+      <inertia ixx="3.97e-05" ixy="0" ixz="0" iyy="3.97e-05" iyz="0" izz="5.83e-05"/>
     </inertial>
     <!-- Part axis5 -->
@@ -2148,5 +2148,5 @@
       <origin xyz="-0.02 -0.02 -0.025" rpy="1.5708 -0 -0"/>
       <geometry>
-        <mesh filename="package://robot_description1/meshes/axis5.stl"/>
+        <box size="0.05 0.05 0.03"/>
       </geometry>
     </collision>
@@ -2156,6 +2156,6 @@
     <inertial>
       <origin xyz="0 0 0" rpy="0 0 0"/>
-      <mass value="1e-09"/>
-      <inertia ixx="1e-09" ixy="0" ixz="0" iyy="1e-09" iyz="0" izz="1e-09"/>
+      <mass value="0.10"/>
+      <inertia ixx="1.50e-05" ixy="0" ixz="0" iyy="2.08e-05" iyz="0" izz="2.08e-05"/>
     </inertial>
     <!-- Part axis6 -->
@@ -2172,5 +2172,5 @@
       <origin xyz="-0.02 0.005 -0.015" rpy="-0 -0 0"/>
       <geometry>
-        <mesh filename="package://robot_description1/meshes/axis6.stl"/>
+        <box size="0.04 0.03 0.03"/>
       </geometry>
     </collision>
@@ -2228,6 +2228,6 @@
     <inertial>
       <origin xyz="0 0 0" rpy="0 0 0"/>
-      <mass value="1e-09"/>
-      <inertia ixx="1e-09" ixy="0" ixz="0" iyy="1e-09" iyz="0" izz="1e-09"/>
+      <mass value="0.25"/>
+      <inertia ixx="8.33e-05" ixy="0" ixz="0" iyy="8.33e-05" iyz="0" izz="1.50e-04"/>
     </inertial>
     <!-- Part axis1_3 -->
@@ -2244,5 +2244,5 @@
       <origin xyz="0.028783 -0.00982538 -0.01" rpy="0 -0 2.97778"/>
       <geometry>
-        <mesh filename="package://robot_description1/meshes/axis1.stl"/>
+        <box size="0.06 0.06 0.02"/>
       </geometry>
     </collision>
@@ -2252,6 +2252,6 @@
     <inertial>
       <origin xyz="0 0 0" rpy="0 0 0"/>
-      <mass value="1e-09"/>
-      <inertia ixx="1e-09" ixy="0" ixz="0" iyy="1e-09" iyz="0" izz="1e-09"/>
+      <mass value="0.20"/>
+      <inertia ixx="5.67e-05" ixy="0" ixz="0" iyy="5.67e-05" iyz="0" izz="8.33e-05"/>
     </inertial>
     <!-- Part axis2_2 -->
@@ -2268,5 +2268,5 @@
       <origin xyz="-0.025 -0.025 -0.015" rpy="1.5708 0 -0"/>
       <geometry>
-        <mesh filename="package://robot_description1/meshes/axis2.stl"/>
+        <box size="0.05 0.05 0.03"/>
       </geometry>
     </collision>
@@ -2276,6 +2276,6 @@
     <inertial>
       <origin xyz="0 0 0" rpy="0 0 0"/>
-      <mass value="1e-09"/>
-      <inertia ixx="1e-09" ixy="0" ixz="0" iyy="1e-09" iyz="0" izz="1e-09"/>
+      <mass value="0.18"/>
+      <inertia ixx="4.80e-05" ixy="0" ixz="0" iyy="6.15e-05" iyz="0" izz="6.15e-05"/>
     </inertial>
     <!-- Part axis3_2 -->
@@ -2292,5 +2292,5 @@
       <origin xyz="-0.0201356 0.02 0.025" rpy="-1.5708 -0 0"/>
       <geometry>
-        <mesh filename="package://robot_description1/meshes/axis3.stl"/>
+        <box size="0.05 0.04 0.04"/>
       </geometry>
     </collision>
@@ -2300,6 +2300,6 @@
     <inertial>
       <origin xyz="0 0 0" rpy="0 0 0"/>
-      <mass value="1e-09"/>
-      <inertia ixx="1e-09" ixy="0" ixz="0" iyy="1e-09" iyz="0" izz="1e-09"/>
+      <mass value="0.15"/>
+      <inertia ixx="3.13e-05" ixy="0" ixz="0" iyy="4.25e-05" iyz="0" izz="5.13e-05"/>
     </inertial>
     <!-- Part axis4_2 -->
@@ -2316,5 +2316,5 @@
       <origin xyz="-0.02 0.005 -0.02" rpy="0 -0 0"/>
       <geometry>
-        <mesh filename="package://robot_description1/meshes/axis4.stl"/>
+        <box size="0.05 0.04 0.03"/>
       </geometry>
     </collision>
@@ -2324,6 +2324,6 @@
     <inertial>
       <origin xyz="0 0 0" rpy="0 0 0"/>
-      <mass value="1e-09"/>
-      <inertia ixx="1e-09" ixy="0" ixz="0" iyy="1e-09" iyz="0" izz="1e-09"/>
+      <mass value="0.14"/>
+      <inertia ixx="3.97e-05" ixy="0" ixz="0" iyy="3.97e-05" iyz="0" izz="5.83e-05"/>
     </inertial>
     <!-- Part axis5_2 -->
@@ -2340,5 +2340,5 @@
       <origin xyz="-0.02 -0.02 -0.025" rpy="1.5708 -0 -0"/>
       <geometry>
-        <mesh filename="package://robot_description1/meshes/axis5.stl"/>
+        <box size="0.05 0.05 0.03"/>
       </geometry>
     </collision>
@@ -2348,6 +2348,6 @@
     <inertial>
       <origin xyz="0 0 0" rpy="0 0 0"/>
-      <mass value="1e-09"/>
-      <inertia ixx="1e-09" ixy="0" ixz="0" iyy="1e-09" iyz="0" izz="1e-09"/>
+      <mass value="0.10"/>
+      <inertia ixx="1.50e-05" ixy="0" ixz="0" iyy="2.08e-05" iyz="0" izz="2.08e-05"/>
     </inertial>
     <!-- Part axis6_2 -->
@@ -2364,5 +2364,5 @@
       <origin xyz="-0.02 0.005 -0.015" rpy="-0 -0 -0"/>
       <geometry>
-        <mesh filename="package://robot_description1/meshes/axis6.stl"/>
+        <box size="0.04 0.03 0.03"/>
       </geometry>
     </collision>
@@ -2420,6 +2420,6 @@
     <inertial>
       <origin xyz="0 0 0" rpy="0 0 0"/>
-      <mass value="1e-09"/>
-      <inertia ixx="1e-09" ixy="0" ixz="0" iyy="1e-09" iyz="0" izz="1e-09"/>
+      <mass value="0.25"/>
+      <inertia ixx="8.33e-05" ixy="0" ixz="0" iyy="8.33e-05" iyz="0" izz="1.50e-04"/>
     </inertial>
     <!-- Part axis1_4 -->
@@ -2436,5 +2436,5 @@
       <origin xyz="-0.005 -0.03 -0.01" rpy="0 0 1.5708"/>
       <geometry>
-        <mesh filename="package://robot_description1/meshes/axis1.stl"/>
+        <box size="0.06 0.06 0.02"/>
       </geometry>
     </collision>
@@ -2444,6 +2444,6 @@
     <inertial>
       <origin xyz="0 0 0" rpy="0 0 0"/>
-      <mass value="1e-09"/>
-      <inertia ixx="1e-09" ixy="0" ixz="0" iyy="1e-09" iyz="0" izz="1e-09"/>
+      <mass value="0.20"/>
+      <inertia ixx="5.67e-05" ixy="0" ixz="0" iyy="5.67e-05" iyz="0" izz="8.33e-05"/>
     </inertial>
     <!-- Part axis2_3 -->
@@ -2460,5 +2460,5 @@
       <origin xyz="-0.025 -0.025 -0.015" rpy="1.5708 -0 0"/>
       <geometry>
-        <mesh filename="package://robot_description1/meshes/axis2.stl"/>
+        <box size="0.05 0.05 0.03"/>
       </geometry>
     </collision>
@@ -2468,6 +2468,6 @@
     <inertial>
       <origin xyz="0 0 0" rpy="0 0 0"/>
-      <mass value="1e-09"/>
-      <inertia ixx="1e-09" ixy="0" ixz="0" iyy="1e-09" iyz="0" izz="1e-09"/>
+      <mass value="0.18"/>
+      <inertia ixx="4.80e-05" ixy="0" ixz="0" iyy="6.15e-05" iyz="0" izz="6.15e-05"/>
     </inertial>
     <!-- Part axis3_3 -->
@@ -2484,5 +2484,5 @@
       <origin xyz="-0.0201356 0.02 0.025" rpy="-1.5708 -0 -0"/>
       <geometry>
-        <mesh filename="package://robot_description1/meshes/axis3.stl"/>
+        <box size="0.05 0.04 0.04"/>
       </geometry>
     </collision>
@@ -2492,6 +2492,6 @@
     <inertial>
       <origin xyz="0 0 0" rpy="0 0 0"/>
-      <mass value="1e-09"/>
-      <inertia ixx="1e-09" ixy="0" ixz="0" iyy="1e-09" iyz="0" izz="1e-09"/>
+      <mass value="0.15"/>
+      <inertia ixx="3.13e-05" ixy="0" ixz="0" iyy="4.25e-05" iyz="0" izz="5.13e-05"/>
     </inertial>
     <!-- Part axis4_3 -->
@@ -2508,5 +2508,5 @@
       <origin xyz="-0.02 0.005 -0.02" rpy="-0 -0 0"/>
       <geometry>
-        <mesh filename="package://robot_description1/meshes/axis4.stl"/>
+        <box size="0.05 0.04 0.03"/>
       </geometry>
     </collision>
@@ -2516,6 +2516,6 @@
     <inertial>
       <origin xyz="0 0 0" rpy="0 0 0"/>
-      <mass value="1e-09"/>
-      <inertia ixx="1e-09" ixy="0" ixz="0" iyy="1e-09" iyz="0" izz="1e-09"/>
+      <mass value="0.14"/>
+      <inertia ixx="3.97e-05" ixy="0" ixz="0" iyy="3.97e-05" iyz="0" izz="5.83e-05"/>
     </inertial>
     <!-- Part axis5_3 -->
@@ -2532,5 +2532,5 @@
       <origin xyz="-0.02 -0.02 -0.025" rpy="1.5708 0 0"/>
       <geometry>
-        <mesh filename="package://robot_description1/meshes/axis5.stl"/>
+        <box size="0.05 0.05 0.03"/>
       </geometry>
     </collision>
@@ -2540,6 +2540,6 @@
     <inertial>
       <origin xyz="0 0 0" rpy="0 0 0"/>
-      <mass value="1e-09"/>
-      <inertia ixx="1e-09" ixy="0" ixz="0" iyy="1e-09" iyz="0" izz="1e-09"/>
+      <mass value="0.10"/>
+      <inertia ixx="1.50e-05" ixy="0" ixz="0" iyy="2.08e-05" iyz="0" izz="2.08e-05"/>
     </inertial>
     <!-- Part axis6_3 -->
@@ -2556,5 +2556,5 @@
       <origin xyz="-0.02 0.005 -0.015" rpy="-0 -0 0"/>
       <geometry>
-        <mesh filename="package://robot_description1/meshes/axis6.stl"/>
+        <box size="0.04 0.03 0.03"/>
       </geometry>
     </collision>
@@ -2618,6 +2618,6 @@
     <inertial>
       <origin xyz="0 0 0" rpy="0 0 0"/>
-      <mass value="1e-09"/>
-      <inertia ixx="1e-09" ixy="0" ixz="0" iyy="1e-09" iyz="0" izz="1e-09"/>
+      <mass value="0.20"/>
+      <inertia ixx="5.67e-05" ixy="0" ixz="0" iyy="5.67e-05" iyz="0" izz="8.33e-05"/>
     </inertial>
     <!-- Part axis2_4 -->
@@ -2634,5 +2634,5 @@
       <origin xyz="-0.025 -0.025 -0.015" rpy="1.5708 0 0"/>
       <geometry>
-        <mesh filename="package://robot_description1/meshes/axis2.stl"/>
+        <box size="0.05 0.05 0.03"/>
       </geometry>
     </collision>
@@ -2642,6 +2642,6 @@
     <inertial>
       <origin xyz="0 0 0" rpy="0 0 0"/>
-      <mass value="1e-09"/>
-      <inertia ixx="1e-09" ixy="0" ixz="0" iyy="1e-09" iyz="0" izz="1e-09"/>
+      <mass value="0.18"/>
+      <inertia ixx="4.80e-05" ixy="0" ixz="0" iyy="6.15e-05" iyz="0" izz="6.15e-05"/>
     </inertial>
     <!-- Part axis3_4 -->
@@ -2658,5 +2658,5 @@
       <origin xyz="-0.0201356 0.02 0.025" rpy="-1.5708 -0 0"/>
       <geometry>
-        <mesh filename="package://robot_description1/meshes/axis3.stl"/>
+        <box size="0.05 0.04 0.04"/>
       </geometry>
     </collision>
@@ -2666,6 +2666,6 @@
     <inertial>
       <origin xyz="0 0 0" rpy="0 0 0"/>
-      <mass value="1e-09"/>
-      <inertia ixx="1e-09" ixy="0" ixz="0" iyy="1e-09" iyz="0" izz="1e-09"/>
+      <mass value="0.15"/>
+      <inertia ixx="3.13e-05" ixy="0" ixz="0" iyy="4.25e-05" iyz="0" izz="5.13e-05"/>
     </inertial>
     <!-- Part axis4_4 -->
@@ -2682,5 +2682,5 @@
       <origin xyz="-0.02 0.005 -0.02" rpy="0 0 -0"/>
       <geometry>
-        <mesh filename="package://robot_description1/meshes/axis4.stl"/>
+        <box size="0.05 0.04 0.03"/>
       </geometry>
     </collision>
@@ -2690,6 +2690,6 @@
     <inertial>
       <origin xyz="0 0 0" rpy="0 0 0"/>
-      <mass value="1e-09"/>
-      <inertia ixx="1e-09" ixy="0" ixz="0" iyy="1e-09" iyz="0" izz="1e-09"/>
+      <mass value="0.14"/>
+      <inertia ixx="3.97e-05" ixy="0" ixz="0" iyy="3.97e-05" iyz="0" izz="5.83e-05"/>
     </inertial>
     <!-- Part axis5_4 -->
@@ -2706,5 +2706,5 @@
       <origin xyz="-0.02 -0.02 -0.025" rpy="1.5708 0 0"/>
       <geometry>
-        <mesh filename="package://robot_description1/meshes/axis5.stl"/>
+        <box size="0.05 0.05 0.03"/>
       </geometry>
     </collision>
@@ -2714,6 +2714,6 @@
     <inertial>
       <origin xyz="0 0 0" rpy="0 0 0"/>
-      <mass value="1e-09"/>
-      <inertia ixx="1e-09" ixy="0" ixz="0" iyy="1e-09" iyz="0" izz="1e-09"/>
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
Commit message: Make z-axis keep its current position defying gravity

File: src/robot_description1/urdf/robot.urdf.xacro (robot description, xacro)
@@ -2030,6 +2030,85 @@
     <child link="leadscrew"/>
     <axis xyz="0 0 -1"/>
+    <dynamics damping="25.0" friction="2.0"/>
     <limit effort="10" velocity="10" lower="-1" upper="1"/>
   </joint>
+  <gazebo reference="leadscrew">
+    <gravity>false</gravity>
+  </gazebo>
+  <gazebo reference="axis1">
+    <gravity>false</gravity>
+  </gazebo>
+  <gazebo reference="axis1_2">
+    <gravity>false</gravity>
+  </gazebo>
+  <gazebo reference="axis2">
+    <gravity>false</gravity>
+  </gazebo>
+  <gazebo reference="axis3">
+    <gravity>false</gravity>
+  </gazebo>
+  <gazebo reference="axis4">
+    <gravity>false</gravity>
+  </gazebo>
+  <gazebo reference="axis5">
+    <gravity>false</gravity>
+  </gazebo>
+  <gazebo reference="axis6">
+    <gravity>false</gravity>
+  </gazebo>
+  <gazebo reference="axis1_3">
+    <gravity>false</gravity>
+  </gazebo>
+  <gazebo reference="axis2_2">
+    <gravity>false</gravity>
+  </gazebo>
+  <gazebo reference="axis3_2">
+    <gravity>false</gravity>
+  </gazebo>
+  <gazebo reference="axis4_2">
+    <gravity>false</gravity>
+  </gazebo>
+  <gazebo reference="axis5_2">
+    <gravity>false</gravity>
+  </gazebo>
+  <gazebo reference="axis6_2">
+    <gravity>false</gravity>
+  </gazebo>
+  <gazebo reference="axis1_4">
+    <gravity>false</gravity>
+  </gazebo>
+  <gazebo reference="axis2_3">
+    <gravity>false</gravity>
+  </gazebo>
+  <gazebo reference="axis3_3">
+    <gravity>false</gravity>
+  </gazebo>
+  <gazebo reference="axis4_3">
+    <gravity>false</gravity>
+  </gazebo>
+  <gazebo reference="axis5_3">
+    <gravity>false</gravity>
+  </gazebo>
+  <gazebo reference="axis6_3">
+    <gravity>false</gravity>
+  </gazebo>
+  <gazebo reference="axis2_4">
+    <gravity>false</gravity>
+  </gazebo>
+  <gazebo reference="axis3_4">
+    <gravity>false</gravity>
+  </gazebo>
+  <gazebo reference="axis4_4">
+    <gravity>false</gravity>
+  </gazebo>
+  <gazebo reference="axis5_4">
+    <gravity>false</gravity>
+  </gazebo>
+  <gazebo reference="axis6_4">
+    <gravity>false</gravity>
+  </gazebo>
+  <gazebo reference="z_bottom_camera_link">
+    <gravity>false</gravity>
+  </gazebo>
   <!-- Link axis1_2 -->
   <link name="axis1_2">
